Commit message: Robot arm works in rviz2

File: src/articubot_one/description/lidar.xacro (robot description, xacro)
@@ -4,5 +4,5 @@
         <parent link="chassis"/>
         <child link="laser_frame"/>
-        <origin xyz="0.122 0 0.212" rpy="0 0 0"/>
+        <origin xyz="0.19 0 0.212" rpy="0 0 0"/>
     </joint>
     <link name="laser_frame">
@@ -11,5 +11,5 @@
                 <cylinder radius="0.05" length="0.04"/>
             </geometry>
-            <material name="black"/>
+            <material name="yellow"/>
         </visual>
         <visual>
@@ -18,5 +18,5 @@
                 <cylinder radius="0.01" length="0.1"/>
             </geometry>
-            <material name="black"/>
+            <material name="yellow"/>
         </visual>
         <collision>
@@ -30,5 +30,5 @@
     </link>
     <gazebo reference="laser_frame">
-        <material>Gazebo/Black</material>
+        <material>Gazebo/Yellow</material>
         <sensor name="laser" type="ray">
             <pose> 0 0 0 0 0 0 </pose>

File: src/articubot_one/description/robot.urdf.xacro (robot description, xacro)
@@ -13,4 +13,5 @@
     <xacro:include filename="camera.xacro" />
     <xacro:include filename="imu.xacro" />
+    <xacro:include filename="robot_arm.urdf" />
     <!-- <xacro:include filename="depth_camera.xacro" /> -->
     <xacro:include filename="face.xacro" />

File: src/articubot_one/description/robot_core.xacro (robot description, xacro)
@@ -33,4 +33,7 @@
     <material name="yellow">
         <color rgba="1 1 0 1"/>
+    </material>
+    <material name="green">
+        <color rgba="0 1 0 1"/>
     </material>
     <!-- BASE LINK -->
