Commit message: Shorter arm

File: src/articubot_one/description/rrbot.urdf.xacro (robot description, xacro)
@@ -12,5 +12,5 @@
   <!-- <xacro:include filename="$(find ros2_control_demo_example_1)/urdf/rrbot.materials.xacro" /> -->
   <!-- Import RRBot ros2_control description -->
-  <!-- <xacro:include filename="$(find articubot_one)/description/rrbot.ros2_control.xacro" /> -->
+  <xacro:include filename="$(find articubot_one)/description/rrbot.ros2_control.xacro" />
   <!-- Used for fixing robot -->
   <!-- <link name="world"/> -->

File: src/articubot_one/description/rrbot_description.urdf.xacro (robot description, xacro)
@@ -3,9 +3,9 @@
   <xacro:macro name="rrbot" params="parent prefix *origin">
   <!-- Constants for robot dimensions -->
-  <xacro:property name="mass" value="0.01" /> <!-- arbitrary value for mass -->
-  <xacro:property name="width" value="0.1" /> <!-- Square dimensions (widthxwidth) of beams -->
-  <xacro:property name="height1" value="2" /> <!-- Link 1 -->
-  <xacro:property name="height2" value="1" /> <!-- Link 2 -->
-  <xacro:property name="height3" value="1" /> <!-- Link 3 -->
+  <xacro:property name="mass" value="0.01" />        <!-- arbitrary value for mass -->
+  <xacro:property name="width" value="0.1" />        <!-- Square dimensions (widthxwidth) of beams -->
+  <xacro:property name="height1" value="1.00" />     <!-- Link 1 -->
+  <xacro:property name="height2" value="0.50" />     <!-- Link 2 -->
+  <xacro:property name="height3" value="0.50" />     <!-- Link 3 -->
   <xacro:property name="axel_offset" value="0.05" /> <!-- Space btw top of beam and the each joint -->
   <joint name="${prefix}base_joint" type="fixed">
@@ -69,5 +69,5 @@
         </inertial>
       </link>
-      <joint name="${prefix}joint2" type="fixed"> <!-- continuous">  -->
+      <joint name="${prefix}joint2" type="continuous">
         <parent link="${prefix}link1"/>
         <child link="${prefix}link2"/>
@@ -107,5 +107,5 @@
       </gazebo>
       <gazebo reference="${prefix}link2">
-        <material>Gazebo/Blue</material>
+        <material>Gazebo/Purple</material>
       </gazebo>
   </xacro:macro>
