Commit message: Real robot messages get thru

File: src/articubot_one/description/rrbot_description.urdf.xacro (robot description, xacro)
@@ -12,8 +12,8 @@
     <xacro:insert_block name="origin" />
     <parent link="${parent}"/>
-    <child link="arm_base_link" />
+    <child link="base_link_arm" />
   </joint>
   <!-- Base Link -->
-  <link name="arm_base_link">
+  <link name="base_link_arm">
     <collision>
       <origin xyz="0 0 ${height1/2}" rpy="0 0 0"/>
@@ -39,5 +39,5 @@
     </link>
     <joint name="${prefix}joint1" type="continuous">
-      <parent link="arm_base_link"/>
+      <parent link="base_link_arm"/>
       <child link="${prefix}link1"/>
       <origin xyz="0 ${width} ${height1 - axel_offset}" rpy="0 0 0"/>
@@ -100,5 +100,5 @@
           </inertial>
         </link>
-      <gazebo reference="arm_base_link">
+      <gazebo reference="base_link_arm">
         <material>Gazebo/Green</material>
       </gazebo>

Commit message: Time to fix this arm

File: src/articubot_one/description/rrbot_description.urdf.xacro (robot description, xacro)
@@ -2,111 +2,111 @@
 <robot xmlns:xacro="http://www.ros.org/wiki/xacro">
   <xacro:macro name="rrbot" params="parent prefix *origin">
-  <!-- Constants for robot dimensions -->
-  <xacro:property name="mass" value="0.01" />        <!-- arbitrary value for mass -->
-  <xacro:property name="width" value="0.1" />        <!-- Square dimensions (widthxwidth) of beams -->
-  <xacro:property name="height1" value="1.00" />     <!-- Link 1 -->
-  <xacro:property name="height2" value="0.50" />     <!-- Link 2 -->
-  <xacro:property name="height3" value="0.50" />     <!-- Link 3 -->
-  <xacro:property name="axel_offset" value="0.05" /> <!-- Space btw top of beam and the each joint -->
-  <joint name="base_joint_arm" type="fixed">
-    <xacro:insert_block name="origin" />
-    <parent link="${parent}"/>
-    <child link="base_link_arm" />
-  </joint>
-  <!-- Base Link -->
-  <link name="base_link_arm">
-    <collision>
-      <origin xyz="0 0 ${height1/2}" rpy="0 0 0"/>
-      <geometry>
-        <box size="${width} ${width} ${height1}"/>
-      </geometry>
-    </collision>
-    <visual>
-      <origin xyz="0 0 ${height1/2}" rpy="0 0 0"/>
-      <geometry>
-        <box size="${width} ${width} ${height1}"/>
-      </geometry>
-      <material name="green"/>
-    </visual>
-    <inertial>
-      <origin xyz="0 0 ${height1/2}" rpy="0 0 0"/>
-      <mass value="${mass}"/>
-      <inertia
-        ixx="${mass / 12.0 * (width*width + height1*height1)}" ixy="0.0" ixz="0.0"
-        iyy="${mass / 12.0 * (height1*height1 + width*width)}" iyz="0.0"
-        izz="${mass / 12.0 * (width*width + width*width)}"/>
-      </inertial>
-    </link>
-    <joint name="${prefix}joint1" type="fixed">
-      <parent link="base_link_arm"/>
-      <child link="${prefix}link1"/>
-      <origin xyz="0 ${width} ${height1 - axel_offset}" rpy="0 0 0"/>
-      <axis xyz="0 1 0"/>
-      <dynamics damping="0.7"/>
+    <!-- Constants for robot dimensions -->
+    <xacro:property name="mass" value="0.01" />        <!-- arbitrary value for mass -->
+    <xacro:property name="width" value="0.1" />        <!-- Square dimensions (widthxwidth) of beams -->
+    <xacro:property name="height1" value="1.0" />      <!-- Link 1 -->
+    <xacro:property name="height2" value="0.5" />     <!-- Link 2 -->
+    <xacro:property name="height3" value="0.5" />     <!-- Link 3 -->
+    <xacro:property name="axel_offset" value="0.05" /> <!-- Space btw top of beam and the each joint -->
+    <!-- Base Link -->
+    <joint name="base_joint_arm" type="fixed">
+      <xacro:insert_block name="origin" />
+      <parent link="${parent}" />
+      <child link="base_link_arm" />
     </joint>
-    <!-- Middle Link -->
-    <link name="${prefix}link1">
+    <link name="base_link_arm">
       <collision>
-        <origin xyz="0 0 ${height2/2 - axel_offset}" rpy="0 0 0"/>
+        <origin xyz="0 0 ${height1/2}" rpy="0 0 0" />
         <geometry>
-          <box size="${width} ${width} ${height2}"/>
+          <box size="${width} ${width} ${height1}" />
         </geometry>
       </collision>
       <visual>
-        <origin xyz="0 0 ${height2/2 - axel_offset}" rpy="0 0 0"/>
+        <origin xyz="0 0 ${height1/2}" rpy="0 0 0" />
         <geometry>
-          <box size="${width} ${width} ${height2}"/>
+          <box size="${width} ${width} ${height1}" />
         </geometry>
-        <material name="yellow"/>
+        <material name="green" />
       </visual>
       <inertial>
-        <origin xyz="0 0 ${height2/2 - axel_offset}" rpy="0 0 0"/>
-        <mass value="${mass}"/>
+        <origin xyz="0 0 ${height1/2}" rpy="0 0 0" />
+        <mass value="${mass}" />
+        <inertia
+          ixx="${mass / 12.0 * (width*width + height1*height1)}" ixy="0.0" ixz="0.0"
+          iyy="${mass / 12.0 * (height1*height1 + width*width)}" iyz="0.0"
+          izz="${mass / 12.0 * (width*width + width*width)}" />
+      </inertial>
+    </link>
+    <gazebo reference="base_link_arm">
+      <material>Gazebo/Green</material>
+    </gazebo>
+    <!-- Middle Link -->
+    <joint name="${prefix}joint1" type="fixed">
+      <parent link="base_link_arm" />
+      <child link="${prefix}link1" />
+      <origin xyz="0 ${width} ${height1 - axel_offset}" rpy="0 0 0" />
+      <axis xyz="0 1 0" />
+      <dynamics damping="0.7" />
+    </joint>
+    <link name="${prefix}link1">
+      <collision>
+        <origin xyz="0 0 ${height2/2 - axel_offset}" rpy="0 0 0" />
+        <geometry>
+          <box size="${width} ${width} ${height2}" />
+        </geometry>
+      </collision>
+      <visual>
+        <origin xyz="0 0 ${height2/2 - axel_offset}" rpy="0 0 0" />
+        <geometry>
+          <box size="${width} ${width} ${height2}" />
+        </geometry>
+        <material name="yellow" />
+      </visual>
+      <inertial>
+        <origin xyz="0 0 ${height2/2 - axel_offset}" rpy="0 0 0" />
+        <mass value="${mass}" />
         <inertia
           ixx="${mass / 12.0 * (width*width + height2*height2)}" ixy="0.0" ixz="0.0"
           iyy="${mass / 12.0 * (height2*height2 + width*width)}" iyz="0.0"
-          izz="${mass / 12.0 * (width*width + width*width)}"/>
-        </inertial>
-      </link>
-      <joint name="${prefix}joint2" type="continuous">
-        <parent link="${prefix}link1"/>
-        <child link="${prefix}link2"/>
-        <origin xyz="0 ${width} ${height2 - axel_offset*2}" rpy="0 0 0"/>
-        <axis xyz="0 1 0"/>
-        <dynamics damping="0.7"/>
-      </joint>
-      <!-- Top Link -->
-      <link name="${prefix}link2">
-        <collision>
-          <origin xyz="0 0 ${height3/2 - axel_offset}" rpy="0 0 0"/>
-          <geometry>
-            <box size="${width} ${width} ${height3}"/>
-          </geometry>
-        </collision>
-        <visual>
-          <origin xyz="0 0 ${height3/2 - axel_offset}" rpy="0 0 0"/>
-          <geometry>
-            <box size="${width} ${width} ${height3}"/>
-          </geometry>
-          <material name="orange"/>
-        </visual>
-        <inertial>
-          <origin xyz="0 0 ${height3/2 - axel_offset}" rpy="0 0 0"/>
-          <mass value="${mass}"/>
-          <inertia
-            ixx="${mass / 12.0 * (width*width + height3*height3)}" ixy="0.0" ixz="0.0"
-            iyy="${mass / 12.0 * (height3*height3 + width*width)}" iyz="0.0"
-            izz="${mass / 12.0 * (width*width + width*width)}"/>
-          </inertial>
-        </link>
-      <gazebo reference="base_link_arm">
-        <material>Gazebo/Green</material>
-      </gazebo>
-      <gazebo reference="${prefix}link1">
-        <material>Gazebo/Yellow</material>
-      </gazebo>
-      <gazebo reference="${prefix}link2">
-        <material>Gazebo/Orange</material>
-      </gazebo>
+          izz="${mass / 12.0 * (width*width + width*width)}" />
+      </inertial>
+    </link>
+    <gazebo reference="${prefix}link1">
+      <material>Gazebo/Yellow</material>
+    </gazebo>
+    <!-- Top Link -->
+    <joint name="${prefix}joint2" type="continuous">
+      <parent link="${prefix}link1" />
+      <child link="${prefix}link2" />
+      <origin xyz="0 ${width} ${height2 - axel_offset*2}" rpy="0 0 0" />
+      <axis xyz="0 1 0" />
+      <dynamics damping="0.7" />
+    </joint>
+    <link name="${prefix}link2">
+      <collision>
+        <origin xyz="0 0 ${height3/2 - axel_offset}" rpy="0 0 0" />
+        <geometry>
+          <box size="${width} ${width} ${height3}" />
+        </geometry>
+      </collision>
+      <visual>
+        <origin xyz="0 0 ${height3/2 - axel_offset}" rpy="0 0 0" />
+        <geometry>
+          <box size="${width} ${width} ${height3}" />
+        </geometry>
+        <material name="orange" />
+      </visual>
+      <inertial>
+        <origin xyz="0 0 ${height3/2 - axel_offset}" rpy="0 0 0" />
+        <mass value="${mass}" />
+        <inertia
+          ixx="${mass / 12.0 * (width*width + height3*height3)}" ixy="0.0" ixz="0.0"
+          iyy="${mass / 12.0 * (height3*height3 + width*width)}" iyz="0.0"
+          izz="${mass / 12.0 * (width*width + width*width)}" />
+      </inertial>
+    </link>
+    <gazebo reference="${prefix}link2">
+      <material>Gazebo/Orange</material>
+    </gazebo>
   </xacro:macro>
 </robot>
