Commit message: Arm shows up in gazebo but it's unstable

File: src/articubot_one/description/robot_core.xacro (robot description, xacro)
@@ -74,5 +74,5 @@
             </geometry>
         </collision>
-        <xacro:inertial_box mass="0.5" x="${chassis_length}" y="${chassis_width}" z="${chassis_height}">
+        <xacro:inertial_box mass="2.0" x="${chassis_length}" y="${chassis_width}" z="${chassis_height}">
             <origin xyz="${chassis_length/2} 0 ${chassis_height/2}" rpy="0 0 0"/>
         </xacro:inertial_box>

File: src/articubot_one/description/ros2_control.xacro (robot description, xacro)
@@ -99,5 +99,40 @@
                 <state_interface name="position" />
             </joint> -->
+            <joint name="joint1">
+                <command_interface name="position">
+                    <param name="min">-1</param>
+                    <param name="max">1</param>
+                </command_interface>
+                <state_interface name="position" />
+            </joint>
+            <joint name="joint2">
+                <command_interface name="position">
+                    <param name="min">-1</param>
+                    <param name="max">1</param>
+                </command_interface>
+                <state_interface name="position" />
+            </joint>
+            <joint name="joint3">
+                <command_interface name="position">
+                    <param name="min">-1</param>
+                    <param name="max">1</param>
+                </command_interface>
+                <state_interface name="position" />
+            </joint>
             <joint name="joint4">
+                <command_interface name="position">
+                    <param name="min">-1</param>
+                    <param name="max">1</param>
+                </command_interface>
+                <state_interface name="position" />
+            </joint>
+            <joint name="joint51">
+                <command_interface name="position">
+                    <param name="min">-1</param>
+                    <param name="max">1</param>
+                </command_interface>
+                <state_interface name="position" />
+            </joint>
+            <joint name="joint52">
                 <command_interface name="position">
                     <param name="min">-1</param>
