Commit message: Arm works with "fixed"

File: src/articubot_one/description/robot.urdf.xacro (robot description, xacro)
@@ -13,6 +13,7 @@
     <xacro:include filename="camera.xacro" />
     <xacro:include filename="imu.xacro" />
-    <xacro:include filename="robot_arm.urdf" />
+    <xacro:include filename="rrbot.urdf.xacro" />
+    <!-- <xacro:include filename="robot_arm.xacro" />    -->
     <!-- <xacro:include filename="depth_camera.xacro" /> -->
-    <xacro:include filename="face.xacro" />
+    <!-- <xacro:include filename="face.xacro" />         -->
 </robot>

File: src/articubot_one/description/robot_arm.xacro (robot description, xacro)
@@ -1,4 +1,4 @@
 <?xml version="1.0"?>
-<robot xmlns:xacro="http://www.ros.org/wiki/xacro" >
+<robot xmlns:xacro="http://www.ros.org/wiki/xacro">
   <link name="arm_base">
     <inertial>
@@ -21,18 +21,23 @@
         rpy="0 0 0" />
       <geometry>
-      	<mesh filename="file:/home/antonio/Documents/Projects/pinecone_pi4_ws/src/articubot_one/meshes/arm_base.stl" />
-      </geometry>
-      <material name="green"/>
-    </visual>
-    <collision>
-      <origin
-        xyz="0 0 0"
-        rpy="0 0 0" />
-      <geometry>
-     	<mesh filename="file:/home/antonio/Documents/Projects/pinecone_pi4_ws/src/articubot_one/meshes/arm_base.stl" />
-      </geometry>
-    </collision>
-</link>
-<link name="bicep">
+          <cylinder radius="0.05" length="0.04"/>
+          <!--
+        <mesh
+          filename="file:/home/antonio/Documents/Projects/pinecone_pi4_ws/src/articubot_one/meshes/arm_base.dae" />
+-->
+      </geometry>
+      <material name="green" />
+    </visual>
+    <collision>
+      <origin
+        xyz="0 0 0"
+        rpy="0 0 0" />
+      <geometry>
+        <mesh
+          filename="file:/home/antonio/Documents/Projects/pinecone_pi4_ws/src/articubot_one/meshes/arm_base.stl" />
+      </geometry>
+    </collision>
+  </link>
+  <link name="bicep">
     <inertial>
       <origin
@@ -54,14 +59,16 @@
         rpy="0 -1.5708 0" />
       <geometry>
-      	<mesh filename="file:/home/antonio/Documents/Projects/pinecone_pi4_ws/src/articubot_one/meshes/bicep.stl" />
-      </geometry>
-      <material name="green"/>
-    </visual>
-    <collision>
-      <origin
-        xyz="0 0 0"
-        rpy="0 -1.5708 0" />
-      <geometry>
-      	<mesh filename="file:/home/antonio/Documents/Projects/pinecone_pi4_ws/src/articubot_one/meshes/bicep.stl" />
+        <mesh
+          filename="file:/home/antonio/Documents/Projects/pinecone_pi4_ws/src/articubot_one/meshes/bicep.stl" />
+      </geometry>
+      <material name="green" />
+    </visual>
+    <collision>
+      <origin
+        xyz="0 0 0"
+        rpy="0 -1.5708 0" />
+      <geometry>
+        <mesh
+          filename="file:/home/antonio/Documents/Projects/pinecone_pi4_ws/src/articubot_one/meshes/bicep.stl" />
       </geometry>
     </collision>
@@ -88,18 +95,20 @@
         rpy="3.14 0 1.5708" />
       <geometry>
-      	<mesh filename="file:/home/antonio/Documents/Projects/pinecone_pi4_ws/src/articubot_one/meshes/wrist.stl" />
-      </geometry>
-      <material name="green"/>
-    </visual>
-    <collision>
-      <origin
-        xyz="0 0 0.13522"
-        rpy="3.14 0 1.5708" />
-      <geometry>
-      	<mesh filename="file:/home/antonio/Documents/Projects/pinecone_pi4_ws/src/articubot_one/meshes/wrist.stl" />
-      </geometry>
-    </collision>
-  </link>
- <link name="elbow">
+        <mesh
+          filename="file:/home/antonio/Documents/Projects/pinecone_pi4_ws/src/articubot_one/meshes/wrist.stl" />
+      </geometry>
+      <material name="green" />
+    </visual>
+    <collision>
+      <origin
+        xyz="0 0 0.13522"
+        rpy="3.14 0 1.5708" />
+      <geometry>
+        <mesh
+          filename="file:/home/antonio/Documents/Projects/pinecone_pi4_ws/src/articubot_one/meshes/wrist.stl" />
+      </geometry>
+    </collision>
+  </link>
+  <link name="elbow">
     <inertial>
       <origin
@@ -121,7 +130,8 @@
         rpy="0 -1.5708 0" />
       <geometry>
-      	<mesh filename="file:/home/antonio/Documents/Projects/pinecone_pi4_ws/src/articubot_one/meshes/elbow.stl" />
-      </geometry>
-      <material name="green"/>
+        <mesh
+          filename="file:/home/antonio/Documents/Projects/pinecone_pi4_ws/src/articubot_one/meshes/elbow.stl" />
+      </geometry>
+      <material name="green" />
     </visual>
     <collision>
@@ -130,9 +140,10 @@
         rpy="0 -1.5708 0" />
       <geometry>
-      	<mesh filename="file:/home/antonio/Documents/Projects/pinecone_pi4_ws/src/articubot_one/meshes/elbow.stl" />
-      </geometry>
-    </collision>
-  </link>
-<link
+        <mesh
+          filename="file:/home/antonio/Documents/Projects/pinecone_pi4_ws/src/articubot_one/meshes/elbow.stl" />
+      </geometry>
+    </collision>
+  </link>
+  <link
     name="top_wrist">
     <inertial>
@@ -155,49 +166,51 @@
         rpy="3.14 0 1.5708" />
       <geometry>
-     	<mesh filename="file:/home/antonio/Documents/Projects/pinecone_pi4_ws/src/articubot_one/meshes/wrist.stl" />
-      </geometry>
-      <material name="green"/>
-    </visual>
-    <collision>
-      <origin
-        xyz="0 0 0.13522"
-        rpy="3.14 0 1.5708" />
-      <geometry>
-      	<mesh filename="file:/home/antonio/Documents/Projects/pinecone_pi4_ws/src/articubot_one/meshes/wrist.stl" />
-      </geometry>
-    </collision>
-  </link>
-<!--######################################################################-->
-<joint name="arm_base_joint" type="continuous">
-  <axis xyz="0 0 1"/>
-  <parent link="base_link"/>
-  <child link="arm_base"/>
-  <origin xyz="-0.16 0 0.12" rpy="0 0 0"/>
-</joint>
-<joint name="shoulder_joint" type="continuous">
-  <axis xyz="0 1 0"/>
-  <parent link="arm_base"/>
-  <child link="bicep"/>
-  <origin rpy="0 0 1.5708" xyz="-0.05166 0.0 0.20271"/>
-</joint>
-<joint name="bottom_wrist_joint" type="continuous">
-  <axis xyz="0 1 0"/>
-  <parent link="bicep"/>
-  <child link="bottom_wrist"/>
-  <origin rpy="0 0 0" xyz="0.0 -0.05194 0.269"/>
-</joint>
-<joint name="elbow_joint" type="continuous">
-  <axis xyz="0 0 1"/>
-  <parent link="bottom_wrist"/>
-  <child link="elbow"/>
-  <origin rpy="0 0 0" xyz="0.0 0 0.13522"/>
-</joint>
-<joint name="top_wrist_joint" type="continuous">
-  <axis xyz="0 1 0"/>
-  <parent link="elbow"/>
-  <child link="top_wrist"/>
-  <origin rpy="0 0 0" xyz="0.0 0 0.20994"/>
-</joint>
-<!--######################################################################-->
+        <mesh
+          filename="file:/home/antonio/Documents/Projects/pinecone_pi4_ws/src/articubot_one/meshes/wrist.stl" />
+      </geometry>
+      <material name="green" />
+    </visual>
+    <collision>
+      <origin
+        xyz="0 0 0.13522"
+        rpy="3.14 0 1.5708" />
+      <geometry>
+        <mesh
+          filename="file:/home/antonio/Documents/Projects/pinecone_pi4_ws/src/articubot_one/meshes/wrist.stl" />
+      </geometry>
+    </collision>
+  </link>
+  <!--######################################################################-->
+  <joint name="arm_base_joint" type="continuous">
+    <axis xyz="0 0 1" />
+    <parent link="base_link" />
+    <child link="arm_base" />
+    <origin xyz="-0.16 0 0.12" rpy="0 0 0" />
+  </joint>
+  <joint name="shoulder_joint" type="continuous">
+    <axis xyz="0 1 0" />
+    <parent link="arm_base" />
+    <child link="bicep" />
+    <origin rpy="0 0 1.5708" xyz="-0.05166 0.0 0.20271" />
+  </joint>
+  <joint name="bottom_wrist_joint" type="continuous">
+    <axis xyz="0 1 0" />
+    <parent link="bicep" />
+    <child link="bottom_wrist" />
+    <origin rpy="0 0 0" xyz="0.0 -0.05194 0.269" />
+  </joint>
+  <joint name="elbow_joint" type="continuous">
+    <axis xyz="0 0 1" />
+    <parent link="bottom_wrist" />
+    <child link="elbow" />
+    <origin rpy="0 0 0" xyz="0.0 0 0.13522" />
+  </joint>
+  <joint name="top_wrist_joint" type="continuous">
+    <axis xyz="0 1 0" />
+    <parent link="elbow" />
+    <child link="top_wrist" />
+    <origin rpy="0 0 0" xyz="0.0 0 0.20994" />
+  </joint>
+  <!--######################################################################-->
   <gazebo reference="arm_base">
     <material>Gazebo/Green</material>
@@ -215,11 +228,16 @@
     <material>Gazebo/Green</material>
   </gazebo>
-<!--
   <gazebo>
     <plugin name="joint_state_publisher" filename="libgazebo_ros_joint_state_publisher.so">
-      <jointName>arm_base_joint, shoulder_joint, bottom_wrist_joint, elbow_joint, bottom_wrist_joint</jointName>
+      <update_rate>30</update_rate>
+      <joint_name>arm_base_joint</joint_name>
+      <joint_name>shoulder_joint</joint_name>
+      <joint_name>bottom_wrist_joint</joint_name>
+      <joint_name>elbow_joint</joint_name>
+      <joint_name>bottom_wrist_joint</joint_name>
+      <!--
+      -->
     </plugin>
   </gazebo>
--->
-<!--######################################################################-->
+  <!--######################################################################-->
 </robot>

File: src/articubot_one/description/robot_core.xacro (robot description, xacro)
@@ -36,4 +36,10 @@
     <material name="green">
         <color rgba="0 1 0 1"/>
+    </material>
+    <material name="grey">
+        <color rgba="0.2 0.2 0.2 1.0"/>
+    </material>
+    <material name="brown">
+        <color rgba="${222/255} ${207/255} ${195/255} 1.0"/>
     </material>
     <!-- BASE LINK -->

Commit message: Floppy eezybotarm in gazebo

File: src/articubot_one/description/robot.urdf.xacro (robot description, xacro)
@@ -17,4 +17,4 @@
     <!-- <xacro:include filename="rrbot.urdf.xacro" /> -->
     <xacro:include filename="$(find robot_arm)/urdf/robot_arm.urdf" />
-    <xacro:include filename="$(find eezybotarm)/urdf/eezybotarm.urdf" />
+    <xacro:include filename="$(find eezybotarm)/urdf/eezybotarm.urdf.xacro" />
 </robot>

File: src/eezybotarm/urdf/eezybotarm.urdf.xacro (robot description, xacro)
@@ -1,4 +1,4 @@
 <?xml version="1.0"?>
-<robot name="eezybotarm">
+<robot xmlns:xacro="http://www.ros.org/wiki/xacro"  name="eezybotarm">
 <!-- BASE LINK -->
   <!-- <link name="base_link"></link> -->
@@ -6,5 +6,5 @@
     <parent link="base_link" />
     <child link="base_link_eezybotarm" />
-    <origin xyz="-0.14 0 0.13" rpy="0 0 0" />
+    <origin xyz="-0.12 -0.09 0.13" rpy="0 0 0" />
   </joint>
   <link
@@ -13,5 +13,5 @@
       <origin xyz="0 0 0" rpy="0 0 0" />
       <geometry>
-        <mesh filename="package://eezybotarm/meshes/base_link_eezybotarm.STL" />
+        <mesh filename="file://$(find eezybotarm)/meshes/base_link.STL" />
       </geometry>
       <material name="">
@@ -25,4 +25,7 @@
       <origin rpy="0 0 0" xyz="0 0 0"/>
     </collision>
+    <xacro:inertial_box mass="0.1" x="0.1" y="0.1" z="0.1">
+      <origin xyz="0 0 0" rpy="0 0 0"/>
+    </xacro:inertial_box>
   </link>
 <!-- JOINT 1 HIP-->
@@ -42,5 +45,5 @@
         xyz="0 -0.04 0" rpy="0 0 0" />
       <geometry>
-        <mesh filename="package://eezybotarm/meshes/link_1.STL" />
+        <mesh filename="file://$(find eezybotarm)/meshes/link_1.STL" />
       </geometry>
       <material name="">
@@ -52,7 +55,10 @@
         xyz="0 -0.04 0" rpy="0 0 0" />
       <geometry>
-        <mesh filename="package://eezybotarm/meshes/link_1.STL" />
-      </geometry>
-    </collision>
+        <mesh filename="file://$(find eezybotarm)/meshes/link_1.STL" />
+      </geometry>
+    </collision>
+    <xacro:inertial_box mass="0.01" x="0.01" y="0.01" z="0.01">
+      <origin xyz="0 0 0" rpy="0 0 0"/>
+    </xacro:inertial_box>
   </link>
 <!-- JOINT 2 SHOULDER -->
@@ -70,5 +76,5 @@
       <origin xyz="0 0 0.0075" rpy="3.14159 0 0" />
       <geometry>
-        <mesh filename="package://eezybotarm/meshes/link_2.STL" />
+        <mesh filename="file://$(find eezybotarm)/meshes/link_2.STL" />
       </geometry>
       <material name="">
@@ -79,7 +85,10 @@
       <origin xyz="0 0 0.0075" rpy="3.14159 0 0" />
       <geometry>
-        <mesh filename="package://eezybotarm/meshes/link_2.STL" />
-      </geometry>
-    </collision>
+        <mesh filename="file://$(find eezybotarm)/meshes/link_2.STL" />
+      </geometry>
+    </collision>
+    <xacro:inertial_box mass="0.05" x="0.1" y="0.1" z="0.1">
+      <origin xyz="0 0 0" rpy="0 0 0"/>
+    </xacro:inertial_box>
   </link>
   <!-- VIRTUAL MIMIC JOINT 2-->
@@ -108,4 +117,7 @@
       <origin rpy="0 0 0" xyz="0 0 0"/>
     </collision>
+    <xacro:inertial_box mass="0.02" x="0.1" y="0.1" z="0.1">
+      <origin xyz="0 0 0" rpy="0 0 0"/>
+    </xacro:inertial_box>
   </link>
 <!-- JOINT 3 ELBOW -->
@@ -123,5 +135,5 @@
       <origin xyz="0 0.0335  0.002" rpy="1.570796325 0 0" />
       <geometry>
-        <mesh filename="package://eezybotarm/meshes/link_3.STL" />
+        <mesh filename="file://$(find eezybotarm)/meshes/link_3.STL" />
       </geometry>
       <material name="">
@@ -132,7 +144,10 @@
       <origin xyz="0 0.0335  0.002" rpy="1.570796325 0 0" />
       <geometry>
-        <mesh filename="package://eezybotarm/meshes/link_3.STL" />
-      </geometry>
-    </collision>
+        <mesh filename="file://$(find eezybotarm)/meshes/link_3.STL" />
+      </geometry>
+    </collision>
+    <xacro:inertial_box mass="0.02" x="0.1" y="0.1" z="0.1">
+      <origin xyz="0 0 0" rpy="0 0 0"/>
+    </xacro:inertial_box>
   </link>
   <!-- JOINT 4 CLAW SUPPORT -->
@@ -150,5 +165,5 @@
       <origin xyz="-0.006 0 -0.0394" rpy="0 0 0" />
       <geometry>
-        <mesh filename="package://eezybotarm/meshes/link_4.STL" scale="0.001 0.001 0.001" />
+        <mesh filename="file://$(find eezybotarm)/meshes/link_4.STL" scale="0.001 0.001 0.001" />
       </geometry>
       <material name="">
@@ -159,7 +174,10 @@
       <origin xyz="-0.006 0 -0.0394" rpy="0 0 0" />
       <geometry>
-        <mesh filename="package://eezybotarm/meshes/link_4.STL" scale="0.001 0.001 0.001" />
-      </geometry>
-    </collision>
+        <mesh filename="file://$(find eezybotarm)/meshes/link_4.STL" scale="0.001 0.001 0.001" />
+      </geometry>
+    </collision>
+    <xacro:inertial_box mass="0.01" x="0.1" y="0.1" z="0.1">
+      <origin xyz="0 0 0" rpy="0 0 0"/>
+    </xacro:inertial_box>
   </link>
   <!-- JOINT 5 CLAW BASE -->
@@ -175,5 +193,5 @@
       <origin xyz="0 0 0" rpy="0 0 0" />
       <geometry>
-        <mesh filename="package://eezybotarm/meshes/link_5.STL" scale="0.001 0.001 0.001" />
+        <mesh filename="file://$(find eezybotarm)/meshes/link_5.STL" scale="0.001 0.001 0.001" />
       </geometry>
       <material name="">
@@ -184,7 +202,10 @@
       <origin xyz="0 0 0" rpy="0 0 0" />
       <geometry>
-        <mesh filename="package://eezybotarm/meshes/link_5.STL" scale="0.001 0.001 0.001" />
-      </geometry>
-    </collision>
+        <mesh filename="file://$(find eezybotarm)/meshes/link_5.STL" scale="0.001 0.001 0.001" />
+      </geometry>
+    </collision>
+    <xacro:inertial_box mass="0.01" x="0.1" y="0.1" z="0.1">
+      <origin xyz="0 0 0" rpy="0 0 0"/>
+    </xacro:inertial_box>
   </link>
   <!-- FINGERS -->
@@ -208,5 +229,5 @@
       <origin xyz="0.0505 0.000 0" rpy="0 0 2.9" />
       <geometry>
-        <mesh filename="package://eezybotarm/meshes/claw_l.STL" scale="0.001 0.001 0.001" />
+        <mesh filename="file://$(find eezybotarm)/meshes/claw_l.STL" scale="0.001 0.001 0.001" />
       </geometry>
     </visual>
@@ -214,5 +235,5 @@
       <origin xyz="0.0505 0.000 0" rpy="0 0 2.9" />
       <geometry>
-        <mesh filename="package://eezybotarm/meshes/claw_l.STL" scale="0.001 0.001 0.001" />
+        <mesh filename="file://$(find eezybotarm)/meshes/claw_l.STL" scale="0.001 0.001 0.001" />
       </geometry>
     </collision>
@@ -222,5 +243,5 @@
       <origin xyz="0.0488 0.0102 0" rpy="0 0 3.14159" />
       <geometry>
-        <mesh filename="package://eezybotarm/meshes/claw_r.STL" scale="0.001 0.001 0.001" />
+        <mesh filename="file://$(find eezybotarm)/meshes/claw_r.STL" scale="0.001 0.001 0.001" />
       </geometry>
     </visual>
@@ -228,5 +249,5 @@
       <origin xyz="0.0488 0.0102 0" rpy="0 0 3.14159" />
       <geometry>
-        <mesh filename="package://eezybotarm/meshes/claw_r.STL" scale="0.001 0.001 0.001" />
+        <mesh filename="file://$(find eezybotarm)/meshes/claw_r.STL" scale="0.001 0.001 0.001" />
       </geometry>
     </collision>
@@ -279,3 +300,24 @@
     <material>Gazebo/Green</material>
   </gazebo>
+  <gazebo reference="link_2">
+    <material>Gazebo/Green</material>
+  </gazebo>
+  <gazebo reference="link_2v">
+    <material>Gazebo/Green</material>
+  </gazebo>
+  <gazebo reference="link_3">
+    <material>Gazebo/Green</material>
+  </gazebo>
+  <gazebo reference="link_4">
+    <material>Gazebo/Green</material>
+  </gazebo>
+  <gazebo reference="claw_base">
+    <material>Gazebo/Green</material>
+  </gazebo>
+  <gazebo reference="claw_l">
+    <material>Gazebo/Green</material>
+  </gazebo>
+  <gazebo reference="claw_r">
+    <material>Gazebo/Green</material>
+  </gazebo>
 </robot>

Commit message: Copied moveit generated ros_control joints

File: src/articubot_one/description/robot.urdf.xacro (robot description, xacro)
@@ -19,6 +19,3 @@
     <!-- <xacro:include filename="$(find eezybotarm)/urdf/eezybotarm.urdf.xacro" /> -->
     <xacro:include filename="$(find arduino_arm)/urdf/arduino_arm.urdf.xacro" />
-    <xacro:include filename="$(find arduino_arm_config)/config/arduino_arm.ros2_control.xacro" />
-    <xacro:arg name="initial_positions_file" default="$(find arduino_arm_config)/config/initial_positions.yaml" />
-    <!-- <xacro:arduino_arm_ros2_control name="FakeSystem" initial_positions_file="$(arg initial_positions_file)"/> -->
 </robot>

File: src/articubot_one/description/ros2_control.xacro (robot description, xacro)
@@ -92,46 +92,39 @@
                 <state_interface name="position" />
             </joint>
-            <!-- <joint name="base_arduino_arm_joint">
-                <command_interface name="position">
-                    <param name="min">-1</param>
-                    <param name="max">1</param>
-                </command_interface>
-                <state_interface name="position" />
+            <joint name="base_waist_joint">
+                <command_interface name="position"/>
+                <state_interface name="position">
+                  <param name="initial_value">0</param>
+                </state_interface>
+                <state_interface name="velocity"/>
             </joint>
             <joint name="shoulder_joint">
-                <command_interface name="position">
-                    <param name="min">-1</param>
-                    <param name="max">1</param>
-                </command_interface>
-                <state_interface name="position" />
+                <command_interface name="position"/>
+                <state_interface name="position">
+                  <param name="initial_value">0</param>
+                </state_interface>
+                <state_interface name="velocity"/>
             </joint>
             <joint name="elbow_joint">
-                <command_interface name="position">
-                    <param name="min">-1</param>
-                    <param name="max">1</param>
-                </command_interface>
-                <state_interface name="position" />
+                <command_interface name="position"/>
+                <state_interface name="position">
+                  <param name="initial_value">0</param>
+                </state_interface>
+                <state_interface name="velocity"/>
             </joint>
             <joint name="wrist_joint">
-                <command_interface name="position">
-                    <param name="min">-1</param>
-                    <param name="max">1</param>
-                </command_interface>
-                <state_interface name="position" />
+                <command_interface name="position"/>
+                <state_interface name="position">
+                  <param name="initial_value">0</param>
+                </state_interface>
+                <state_interface name="velocity"/>
             </joint>
             <joint name="gripper1_joint">
-                <command_interface name="position">
-                    <param name="min">-1</param>
-                    <param name="max">1</param>
-                </command_interface>
-                <state_interface name="position" />
+                <command_interface name="position"/>
+                <state_interface name="position">
+                  <param name="initial_value">0</param>
+                </state_interface>
+                <state_interface name="velocity"/>
             </joint>
-            <joint name="gripper2_joint">
-                <command_interface name="position">
-                    <param name="min">-1</param>
-                    <param name="max">1</param>
-                </command_interface>
-                <state_interface name="position" />
-            </joint> -->
         </ros2_control>
     </xacro:if>
