Commit message: Trying to use diffdrive_esp32

File: src/articubot_one/description/ros2_control.xacro (robot description, xacro)
@@ -2,5 +2,24 @@
 <robot xmlns:xacro="http://www.ros.org/wiki/xacro">
     <xacro:unless value="$(arg sim_mode)">
-        <ros2_control name="RealRobot" type="system">
+        <xacro:macro name="diffbot_ros2_control" params="name prefix">
+            <ros2_control name="${name}" type="system">
+                <hardware>
+                    <plugin>diffdrive_esp32/DiffBotSystemHardware</plugin>
+                    <param name="example_param_hw_start_duration_sec">0</param>
+                    <param name="example_param_hw_stop_duration_sec">3.0</param>
+                </hardware>
+                <joint name="${prefix}left_wheel_joint">
+                    <command_interface name="velocity" />
+                    <state_interface name="position" />
+                    <state_interface name="velocity" />
+                </joint>
+                <joint name="${prefix}right_wheel_joint">
+                    <command_interface name="velocity" />
+                    <state_interface name="position" />
+                    <state_interface name="velocity" />
+                </joint>
+            </ros2_control>
+        </xacro:macro>
+        <!-- <ros2_control name="RealRobot" type="system">
             <hardware>
                 <plugin>diffdrive_arduino/DiffDriveArduino</plugin>
@@ -29,5 +48,5 @@
                 <state_interface name="position"/>
             </joint>
-        </ros2_control>
+        </ros2_control> -->
     </xacro:unless>
     <xacro:if value="$(arg sim_mode)">
@@ -41,6 +60,6 @@
                     <param name="max">10</param>
                 </command_interface>
-                <state_interface name="velocity"/>
-                <state_interface name="position"/>
+                <state_interface name="velocity" />
+                <state_interface name="position" />
             </joint>
             <joint name="right_wheel_joint">
@@ -49,6 +68,6 @@
                     <param name="max">10</param>
                 </command_interface>
-                <state_interface name="velocity"/>
-                <state_interface name="position"/>
+                <state_interface name="velocity" />
+                <state_interface name="position" />
             </joint>
         </ros2_control>

Commit message: Still not sure how to build a hw interface

File: src/articubot_one/description/ros2_control.xacro (robot description, xacro)
@@ -2,24 +2,5 @@
 <robot xmlns:xacro="http://www.ros.org/wiki/xacro">
     <xacro:unless value="$(arg sim_mode)">
-        <xacro:macro name="diffbot_ros2_control" params="name prefix">
-            <ros2_control name="${name}" type="system">
-                <hardware>
-                    <plugin>diffdrive_esp32/DiffBotSystemHardware</plugin>
-                    <param name="example_param_hw_start_duration_sec">0</param>
-                    <param name="example_param_hw_stop_duration_sec">3.0</param>
-                </hardware>
-                <joint name="${prefix}left_wheel_joint">
-                    <command_interface name="velocity" />
-                    <state_interface name="position" />
-                    <state_interface name="velocity" />
-                </joint>
-                <joint name="${prefix}right_wheel_joint">
-                    <command_interface name="velocity" />
-                    <state_interface name="position" />
-                    <state_interface name="velocity" />
-                </joint>
-            </ros2_control>
-        </xacro:macro>
-        <!-- <ros2_control name="RealRobot" type="system">
+        <ros2_control name="RealRobot" type="system">
             <hardware>
                 <plugin>diffdrive_arduino/DiffDriveArduino</plugin>
@@ -37,6 +18,6 @@
                     <param name="max">10</param>
                 </command_interface>
-                <state_interface name="velocity"/>
-                <state_interface name="position"/>
+                <state_interface name="velocity" />
+                <state_interface name="position" />
             </joint>
             <joint name="right_wheel_joint">
@@ -45,8 +26,8 @@
                     <param name="max">10</param>
                 </command_interface>
-                <state_interface name="velocity"/>
-                <state_interface name="position"/>
+                <state_interface name="velocity" />
+                <state_interface name="position" />
             </joint>
-        </ros2_control> -->
+        </ros2_control>
     </xacro:unless>
     <xacro:if value="$(arg sim_mode)">

File: src/diffdrive_esp32/description/ros2_control/diffbot.ros2_control.xacro (robot description, xacro)
@@ -4,5 +4,5 @@
     <ros2_control name="${name}" type="system">
       <hardware>
-        <plugin>diffdrive_esp32/DiffBotSystemHardware</plugin>
+        <plugin>ros2_control_demo_example_2/DiffBotSystemHardware</plugin>
         <param name="example_param_hw_start_duration_sec">0</param>
         <param name="example_param_hw_stop_duration_sec">3.0</param>

File: src/diffdrive_esp32/description/urdf/diffbot.urdf.xacro (robot description, xacro)
@@ -3,9 +3,9 @@
 <robot xmlns:xacro="http://www.ros.org/wiki/xacro" name="diffdrive_robot">
   <xacro:arg name="prefix" default="" />
-  <xacro:include filename="$(find diffdrive_esp32)/urdf/diffbot_description.urdf.xacro" />
+  <xacro:include filename="$(find ros2_control_demo_example_2)/urdf/diffbot_description.urdf.xacro" />
   <!-- Import Rviz colors -->
-  <xacro:include filename="$(find diffdrive_esp32)/urdf/diffbot.materials.xacro" />
+  <xacro:include filename="$(find ros2_control_demo_example_2)/urdf/diffbot.materials.xacro" />
   <!-- Import diffbot ros2_control description -->
-  <xacro:include filename="$(find diffdrive_esp32)/ros2_control/diffbot.ros2_control.xacro" />
+  <xacro:include filename="$(find ros2_control_demo_example_2)/ros2_control/diffbot.ros2_control.xacro" />
   <xacro:diffbot prefix="$(arg prefix)" />
   <xacro:diffbot_ros2_control

Commit message: diffdrive_esp32 working

File: src/articubot_one/description/ros2_control.xacro (robot description, xacro)
@@ -3,4 +3,21 @@
     <xacro:unless value="$(arg sim_mode)">
         <ros2_control name="RealRobot" type="system">
+            <hardware>
+                <plugin>ros2_control_demo_example_2/DiffBotSystemHardware</plugin>
+                <param name="example_param_hw_start_duration_sec">0</param>
+                <param name="example_param_hw_stop_duration_sec">3.0</param>
+            </hardware>
+            <joint name="left_wheel_joint">
+                <command_interface name="velocity"/>
+                <state_interface name="position" />
+                <state_interface name="velocity" />
+            </joint>
+            <joint name="right_wheel_joint">
+                <command_interface name="velocity"/>
+                <state_interface name="position" />
+                <state_interface name="velocity" />
+            </joint>
+        </ros2_control>
+        <!-- <ros2_control name="RealRobot" type="system">
             <hardware>
                 <plugin>diffdrive_arduino/DiffDriveArduino</plugin>
@@ -29,5 +46,5 @@
                 <state_interface name="position" />
             </joint>
-        </ros2_control>
+        </ros2_control> -->
     </xacro:unless>
     <xacro:if value="$(arg sim_mode)">

Commit message: Added more ros2_controllers

File: src/articubot_one/description/ros2_control.xacro (robot description, xacro)
@@ -9,10 +9,10 @@
             </hardware>
             <joint name="left_wheel_joint">
-                <command_interface name="velocity"/>
+                <command_interface name="velocity" />
                 <state_interface name="position" />
                 <state_interface name="velocity" />
             </joint>
             <joint name="right_wheel_joint">
-                <command_interface name="velocity"/>
+                <command_interface name="velocity" />
                 <state_interface name="position" />
                 <state_interface name="velocity" />
@@ -69,4 +69,26 @@
                 <state_interface name="position" />
             </joint>
+<!--
+            <hardware>
+                <plugin>ros2_control_demo_example_1/RRBotSystemPositionOnlyHardware</plugin>
+                <param name="example_param_hw_start_duration_sec">0</param>
+                <param name="example_param_hw_stop_duration_sec">3.0</param>
+                <param name="example_param_hw_slowdown">100</param>
+            </hardware>
+-->
+            <joint name="arm_joint1">
+                <command_interface name="position">
+                    <param name="min">-1</param>
+                    <param name="max">1</param>
+                </command_interface>
+                <state_interface name="position" />
+            </joint>
+            <joint name="arm_joint2">
+                <command_interface name="position">
+                    <param name="min">-1</param>
+                    <param name="max">1</param>
+                </command_interface>
+                <state_interface name="position" />
+            </joint>
         </ros2_control>
     </xacro:if>

Commit message: Clean up a bit

File: src/articubot_one/description/ros2_control.xacro (robot description, xacro)
@@ -76,6 +76,5 @@
                 <param name="example_param_hw_slowdown">100</param>
             </hardware>
--->
-            <joint name="arm_joint1">
+            <joint name="joint1">
                 <command_interface name="position">
                     <param name="min">-1</param>
@@ -84,5 +83,6 @@
                 <state_interface name="position" />
             </joint>
-            <joint name="arm_joint2">
+-->
+            <joint name="joint2">
                 <command_interface name="position">
                     <param name="min">-1</param>

File: src/articubot_one/description/rrbot.urdf.xacro (robot description, xacro)
@@ -6,5 +6,5 @@
 -->
 <robot xmlns:xacro="http://www.ros.org/wiki/xacro" name="2dof_robot">
-  <xacro:arg name="prefix" default="arm_" />
+  <xacro:arg name="prefix" default="" />
   <!-- Import RRBot macro -->
   <xacro:include filename="$(find articubot_one)/description/rrbot_description.urdf.xacro" />
@@ -12,5 +12,5 @@
   <!-- <xacro:include filename="$(find ros2_control_demo_example_1)/urdf/rrbot.materials.xacro" /> -->
   <!-- Import RRBot ros2_control description -->
-  <xacro:include filename="$(find articubot_one)/description/rrbot.ros2_control.xacro" />
+  <!-- <xacro:include filename="$(find articubot_one)/description/rrbot.ros2_control.xacro" /> -->
   <!-- Used for fixing robot -->
   <!-- <link name="world"/> -->

File: src/articubot_one/description/rrbot_description.urdf.xacro (robot description, xacro)
@@ -9,11 +9,11 @@
   <xacro:property name="height3" value="0.50" />     <!-- Link 3 -->
   <xacro:property name="axel_offset" value="0.05" /> <!-- Space btw top of beam and the each joint -->
-  <joint name="${prefix}base_joint" type="fixed">
+  <joint name="arm_base_joint" type="fixed">
     <xacro:insert_block name="origin" />
     <parent link="${parent}"/>
-    <child link="${prefix}base_link" />
+    <child link="arm_base_link" />
   </joint>
   <!-- Base Link -->
-  <link name="${prefix}base_link">
+  <link name="arm_base_link">
     <collision>
       <origin xyz="0 0 ${height1/2}" rpy="0 0 0"/>
@@ -39,5 +39,5 @@
     </link>
     <joint name="${prefix}joint1" type="fixed"> <!-- continuous">  -->
-      <parent link="${prefix}base_link"/>
+      <parent link="arm_base_link"/>
       <child link="${prefix}link1"/>
       <origin xyz="0 ${width} ${height1 - axel_offset}" rpy="0 0 0"/>
@@ -100,5 +100,5 @@
           </inertial>
         </link>
-      <gazebo reference="${prefix}base_link">
+      <gazebo reference="arm_base_link">
         <material>Gazebo/Green</material>
       </gazebo>

Commit message: Joint_trag starts up

File: src/articubot_one/description/ros2_control.xacro (robot description, xacro)
@@ -69,10 +69,14 @@
                 <state_interface name="position" />
             </joint>
-<!--
+        </ros2_control>
+        <ros2_control name="GazeboSystem_RRBot" type="system">
             <hardware>
+                <plugin>gazebo_ros2_control/GazeboSystem</plugin>
+                <!--
                 <plugin>ros2_control_demo_example_1/RRBotSystemPositionOnlyHardware</plugin>
                 <param name="example_param_hw_start_duration_sec">0</param>
                 <param name="example_param_hw_stop_duration_sec">3.0</param>
                 <param name="example_param_hw_slowdown">100</param>
+                -->
             </hardware>
             <joint name="joint1">
@@ -83,5 +87,4 @@
                 <state_interface name="position" />
             </joint>
--->
             <joint name="joint2">
                 <command_interface name="position">

File: src/articubot_one/description/rrbot_description.urdf.xacro (robot description, xacro)
@@ -38,5 +38,5 @@
       </inertial>
     </link>
-    <joint name="${prefix}joint1" type="fixed"> <!-- continuous">  -->
+    <joint name="${prefix}joint1" type="fixed">
       <parent link="arm_base_link"/>
       <child link="${prefix}link1"/>

Commit message: RealRobotArm works

File: src/articubot_one/description/ros2_control.xacro (robot description, xacro)
@@ -17,4 +17,27 @@
                 <state_interface name="position" />
                 <state_interface name="velocity" />
+            </joint>
+        </ros2_control>
+        <ros2_control name="RealRobotArm" type="system">
+            <hardware>
+                <!-- <plugin>gazebo_ros2_control/GazeboSystem</plugin> -->
+                <plugin>ros2_control_demo_example_1/RRBotSystemPositionOnlyHardware</plugin>
+                <param name="example_param_hw_start_duration_sec">0</param>
+                <param name="example_param_hw_stop_duration_sec">3.0</param>
+                <param name="example_param_hw_slowdown">100</param>
+            </hardware>
+            <joint name="joint1">
+                <command_interface name="position">
+                    <param name="min">-1</param>
+                    <param name="max">1</param>
+                </command_interface>
+                <state_interface name="position" />
+            </joint>
+            <joint name="joint2">
+                <command_interface name="position">
+                    <param name="min">-1</param>
+                    <param name="max">1</param>
+                </command_interface>
+                <state_interface name="position" />
             </joint>
         </ros2_control>
@@ -70,29 +93,4 @@
             </joint>
         </ros2_control>
-        <ros2_control name="GazeboSystem_RRBot" type="system">
-            <hardware>
-                <plugin>gazebo_ros2_control/GazeboSystem</plugin>
-                <!--
-                <plugin>ros2_control_demo_example_1/RRBotSystemPositionOnlyHardware</plugin>
-                <param name="example_param_hw_start_duration_sec">0</param>
-                <param name="example_param_hw_stop_duration_sec">3.0</param>
-                <param name="example_param_hw_slowdown">100</param>
-                -->
-            </hardware>
-            <joint name="joint1">
-                <command_interface name="position">
-                    <param name="min">-1</param>
-                    <param name="max">1</param>
-                </command_interface>
-                <state_interface name="position" />
-            </joint>
-            <joint name="joint2">
-                <command_interface name="position">
-                    <param name="min">-1</param>
-                    <param name="max">1</param>
-                </command_interface>
-                <state_interface name="position" />
-            </joint>
-        </ros2_control>
     </xacro:if>
     <gazebo>

File: src/articubot_one/description/rrbot_description.urdf.xacro (robot description, xacro)
@@ -38,5 +38,5 @@
       </inertial>
     </link>
-    <joint name="${prefix}joint1" type="fixed">
+    <joint name="${prefix}joint1" type="continuous">
       <parent link="arm_base_link"/>
       <child link="${prefix}link1"/>

Commit message: Remove forward_posi controller

File: src/articubot_one/description/ros2_control.xacro (robot description, xacro)
@@ -92,4 +92,18 @@
                 <state_interface name="position" />
             </joint>
+            <joint name="joint1">
+                <command_interface name="position">
+                    <param name="min">-1</param>
+                    <param name="max">1</param>
+                </command_interface>
+                <state_interface name="position" />
+            </joint>
+            <joint name="joint2">
+                <command_interface name="position">
+                    <param name="min">-1</param>
+                    <param name="max">1</param>
+                </command_interface>
+                <state_interface name="position" />
+            </joint>
         </ros2_control>
     </xacro:if>

File: src/articubot_one/description/rrbot_description.urdf.xacro (robot description, xacro)
@@ -38,5 +38,5 @@
       </inertial>
     </link>
-    <joint name="${prefix}joint1" type="continuous">
+    <joint name="${prefix}joint1" type="fixed">
       <parent link="arm_base_link"/>
       <child link="${prefix}link1"/>

Commit message: Arm is twitching

File: src/articubot_one/description/ros2_control.xacro (robot description, xacro)
@@ -92,5 +92,5 @@
                 <state_interface name="position" />
             </joint>
-            <joint name="joint1">
+            <!-- <joint name="joint1">
                 <command_interface name="position">
                     <param name="min">-1</param>
@@ -98,5 +98,5 @@
                 </command_interface>
                 <state_interface name="position" />
-            </joint>
+            </joint> -->
             <joint name="joint2">
                 <command_interface name="position">

File: src/articubot_one/description/rrbot_description.urdf.xacro (robot description, xacro)
@@ -9,5 +9,5 @@
   <xacro:property name="height3" value="0.50" />     <!-- Link 3 -->
   <xacro:property name="axel_offset" value="0.05" /> <!-- Space btw top of beam and the each joint -->
-  <joint name="arm_base_joint" type="fixed">
+  <joint name="base_joint_arm" type="fixed">
     <xacro:insert_block name="origin" />
     <parent link="${parent}"/>
@@ -38,5 +38,5 @@
       </inertial>
     </link>
-    <joint name="${prefix}joint1" type="continuous">
+    <joint name="${prefix}joint1" type="fixed">
       <parent link="base_link_arm"/>
       <child link="${prefix}link1"/>
@@ -104,8 +104,8 @@
       </gazebo>
       <gazebo reference="${prefix}link1">
-        <material>Gazebo/Orange</material>
+        <material>Gazebo/Yellow</material>
       </gazebo>
       <gazebo reference="${prefix}link2">
-        <material>Gazebo/Purple</material>
+        <material>Gazebo/Orange</material>
       </gazebo>
   </xacro:macro>

Commit message: Added damping, renamed files

File: src/articubot_one/description/ros2_control.xacro (robot description, xacro)
@@ -92,11 +92,4 @@
                 <state_interface name="position" />
             </joint>
-            <!-- <joint name="joint1">
-                <command_interface name="position">
-                    <param name="min">-1</param>
-                    <param name="max">1</param>
-                </command_interface>
-                <state_interface name="position" />
-            </joint> -->
             <joint name="joint1">
                 <command_interface name="position">
@@ -147,5 +140,5 @@
             <parameters>$(find articubot_one)/config/my_controllers.yaml</parameters>
             <parameters>$(find articubot_one)/config/gaz_ros2_ctl_use_sim.yaml</parameters>
-            <parameters>$(find articubot_one)/config/rrbot_forward_position_publisher.yaml</parameters>
+            <parameters>$(find articubot_one)/config/forward_position_publisher.yaml</parameters>
         </plugin>
     </gazebo>
