Commit message: Eezybotarm moves around but very shaky

File: src/articubot_one/description/ros2_control.xacro (robot description, xacro)
@@ -134,6 +134,41 @@
                 <state_interface name="position" />
             </joint>
-        </ros2_control>
-    </xacro:if>
+        <joint name="joint_1">
+            <command_interface name="position">
+                <param name="min">-1</param>
+                <param name="max">1</param>
+            </command_interface>
+            <state_interface name="position" />
+        </joint>
+        <joint name="joint_2">
+            <command_interface name="position">
+                <param name="min">-1</param>
+                <param name="max">1</param>
+            </command_interface>
+            <state_interface name="position" />
+        </joint>
+        <joint name="joint_2v">
+            <command_interface name="position">
+                <param name="min">-1</param>
+                <param name="max">1</param>
+            </command_interface>
+            <state_interface name="position" />
+        </joint>
+        <joint name="joint_3">
+            <command_interface name="position">
+                <param name="min">-1</param>
+                <param name="max">1</param>
+            </command_interface>
+            <state_interface name="position" />
+        </joint>
+        <joint name="joint_4">
+            <command_interface name="position">
+                <param name="min">-1</param>
+                <param name="max">1</param>
+            </command_interface>
+            <state_interface name="position" />
+        </joint>
+    </ros2_control>
+</xacro:if>
     <gazebo>
         <plugin name="gazebo_ros2_control" filename="libgazebo_ros2_control.so">

File: src/eezybotarm/urdf/eezybotarm.urdf.xacro (robot description, xacro)
@@ -25,5 +25,5 @@
       <origin rpy="0 0 0" xyz="0 0 0"/>
     </collision>
-    <xacro:inertial_box mass="0.1" x="0.1" y="0.1" z="0.1">
+    <xacro:inertial_box mass="0.01" x="0.1" y="0.1" z="0.1">
       <origin xyz="0 0 0" rpy="0 0 0"/>
     </xacro:inertial_box>
@@ -58,5 +58,5 @@
       </geometry>
     </collision>
-    <xacro:inertial_box mass="0.01" x="0.01" y="0.01" z="0.01">
+    <xacro:inertial_box mass="0.001" x="0.01" y="0.01" z="0.01">
       <origin xyz="0 0 0" rpy="0 0 0"/>
     </xacro:inertial_box>
@@ -88,5 +88,5 @@
       </geometry>
     </collision>
-    <xacro:inertial_box mass="0.05" x="0.1" y="0.1" z="0.1">
+    <xacro:inertial_box mass="0.001" x="0.1" y="0.1" z="0.1">
       <origin xyz="0 0 0" rpy="0 0 0"/>
     </xacro:inertial_box>
@@ -117,5 +117,5 @@
       <origin rpy="0 0 0" xyz="0 0 0"/>
     </collision>
-    <xacro:inertial_box mass="0.02" x="0.1" y="0.1" z="0.1">
+    <xacro:inertial_box mass="0.001" x="0.1" y="0.1" z="0.1">
       <origin xyz="0 0 0" rpy="0 0 0"/>
     </xacro:inertial_box>
@@ -147,5 +147,5 @@
       </geometry>
     </collision>
-    <xacro:inertial_box mass="0.02" x="0.1" y="0.1" z="0.1">
+    <xacro:inertial_box mass="0.001" x="0.1" y="0.1" z="0.1">
       <origin xyz="0 0 0" rpy="0 0 0"/>
     </xacro:inertial_box>
@@ -177,5 +177,5 @@
       </geometry>
     </collision>
-    <xacro:inertial_box mass="0.01" x="0.1" y="0.1" z="0.1">
+    <xacro:inertial_box mass="0.001" x="0.1" y="0.1" z="0.1">
       <origin xyz="0 0 0" rpy="0 0 0"/>
     </xacro:inertial_box>
@@ -205,5 +205,5 @@
       </geometry>
     </collision>
-    <xacro:inertial_box mass="0.01" x="0.1" y="0.1" z="0.1">
+    <xacro:inertial_box mass="0.001" x="0.1" y="0.1" z="0.1">
       <origin xyz="0 0 0" rpy="0 0 0"/>
     </xacro:inertial_box>

Commit message: Time to try moveit on mobile robot

File: src/articubot_one/description/ros2_control.xacro (robot description, xacro)
@@ -1,4 +1,5 @@
 <?xml version="1.0"?>
 <robot xmlns:xacro="http://www.ros.org/wiki/xacro">
+    <!-- <xacro:property name="sim_mode" value="true"/> -->
     <xacro:unless value="$(arg sim_mode)">
         <ros2_control name="RealRobot" type="system">
@@ -27,5 +28,5 @@
                 <param name="example_param_hw_slowdown">100</param>
             </hardware>
-            <joint name="joint1">
+            <!-- <joint name="joint1">
                 <command_interface name="position">
                     <param name="min">-1</param>
@@ -40,5 +41,5 @@
                 </command_interface>
                 <state_interface name="position" />
-            </joint>
+            </joint> -->
         </ros2_control>
     </xacro:unless>

Commit message: Move gz_ros/ros2_controllers out of folder

File: src/articubot_one/description/ros2_control.xacro (robot description, xacro)
@@ -20,5 +20,5 @@
             </joint>
         </ros2_control>
-        <!-- <ros2_control name="RealRobotArm" type="system">
+        <ros2_control name="RealRobotArm" type="system">
             <hardware>
                 <plugin>ros2_control_demo_example_1/RRBotSystemPositionOnlyHardware</plugin>
@@ -27,47 +27,40 @@
                 <param name="example_param_hw_slowdown">100</param>
             </hardware>
-            <joint name="base_arduino_arm_joint">
-                <command_interface name="position">
-                    <param name="min">-1</param>
-                    <param name="max">1</param>
-                </command_interface>
-                <state_interface name="position" />
+            <joint name="base_waist_joint">
+              <command_interface name="position">
+                <param name="min">-1</param>
+                <param name="max">1</param>
+              </command_interface>
+              <state_interface name="position"/>
             </joint>
             <joint name="shoulder_joint">
-                <command_interface name="position">
-                    <param name="min">-1</param>
-                    <param name="max">1</param>
-                </command_interface>
-                <state_interface name="position" />
+              <command_interface name="position">
+                <param name="min">-1</param>
+                <param name="max">1</param>
+              </command_interface>
+              <state_interface name="position"/>
             </joint>
             <joint name="elbow_joint">
-                <command_interface name="position">
-                    <param name="min">-1</param>
-                    <param name="max">1</param>
-                </command_interface>
-                <state_interface name="position" />
+              <command_interface name="position">
+                <param name="min">-1</param>
+                <param name="max">1</param>
+              </command_interface>
+              <state_interface name="position"/>
             </joint>
             <joint name="wrist_joint">
-                <command_interface name="position">
-                    <param name="min">-1</param>
-                    <param name="max">1</param>
-                </command_interface>
-                <state_interface name="position" />
+              <command_interface name="position">
+                <param name="min">-1</param>
+                <param name="max">1</param>
+              </command_interface>
+              <state_interface name="position"/>
             </joint>
             <joint name="gripper1_joint">
-                <command_interface name="position">
-                    <param name="min">-1</param>
-                    <param name="max">1</param>
-                </command_interface>
-                <state_interface name="position" />
+              <command_interface name="position">
+                <param name="min">-1</param>
+                <param name="max">1</param>
+              </command_interface>
+              <state_interface name="position"/>
             </joint>
-            <joint name="gripper2_joint">
-                <command_interface name="position">
-                    <param name="min">-1</param>
-                    <param name="max">1</param>
-                </command_interface>
-                <state_interface name="position" />
-            </joint>
-        </ros2_control> -->
+        </ros2_control>
     </xacro:unless>
     <xacro:if value="$(arg sim_mode)">
