Commit message: Gazebo mesh files work but NOT rviz2

File: src/articubot_one/description/camera.xacro (robot description, xacro)
@@ -4,5 +4,5 @@
         <parent link="chassis"/>
         <child link="camera_link"/>
-        <origin xyz="0.276 0 0.181" rpy="0 0.18 0"/>
+        <origin xyz="0.32 0 0.181" rpy="0 0.18 0"/>
     </joint>
     <link name="camera_link">

File: src/articubot_one/description/imu.xacro (robot description, xacro)
@@ -4,5 +4,5 @@
         <parent link="chassis" />
         <child link="imu_link" />
-        <origin xyz="0.235 0 0.14" rpy="0 0 0"/>
+        <origin xyz="0.28 0 0.14" rpy="0 0 0"/>
     </joint>
     <link name="imu_link">

File: src/articubot_one/description/lidar.xacro (robot description, xacro)
@@ -4,5 +4,5 @@
         <parent link="chassis"/>
         <child link="laser_frame"/>
-        <origin xyz="0.19 0 0.212" rpy="0 0 0"/>
+        <origin xyz="0.235 0 0.212" rpy="0 0 0"/>
     </joint>
     <link name="laser_frame">

File: src/robot_arm/urdf/robot_arm.urdf (robot description, URDF)
Before this commit: robot robot_arm, 7 links, 7 joints
Links:
- link base_link_arm: geometry collision mesh filename=/home/antonio/Documents/Projects/pinecone_pi4_ws/src/robot_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; visual mesh filename=/home/antonio/Documents/Projects/pinecone_pi4_ws/src/robot_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
- link link1: geometry collision mesh filename=/home/antonio/Documents/Projects/pinecone_pi4_ws/src/robot_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; visual mesh filename=/home/antonio/Documents/Projects/pinecone_pi4_ws/src/robot_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
- link link2: geometry collision mesh filename=/home/antonio/Documents/Projects/pinecone_pi4_ws/src/robot_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; visual mesh filename=/home/antonio/Documents/Projects/pinecone_pi4_ws/src/robot_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
- link link3: geometry collision mesh filename=/home/antonio/Documents/Projects/pinecone_pi4_ws/src/robot_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; visual mesh filename=/home/antonio/Documents/Projects/pinecone_pi4_ws/src/robot_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
- link link4: geometry collision mesh filename=/home/antonio/Documents/Projects/pinecone_pi4_ws/src/robot_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; visual mesh filename=/home/antonio/Documents/Projects/pinecone_pi4_ws/src/robot_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
- link link51: geometry collision mesh filename=/home/antonio/Documents/Projects/pinecone_pi4_ws/src/robot_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; visual mesh filename=/home/antonio/Documents/Projects/pinecone_pi4_ws/src/robot_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
- link link52: geometry collision mesh filename=/home/antonio/Documents/Projects/pinecone_pi4_ws/src/robot_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; visual mesh filename=/home/antonio/Documents/Projects/pinecone_pi4_ws/src/robot_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
Joints:
- joint base_joint_arm: origin xyz=-0.15 0 0.13 rpy=0 0 0 -> xyz=-0.14 0 0.13 rpy=0 0 0

Commit message: Works standalong. gaz + mov == NO

File: src/articubot_one/description/camera.xacro (robot description, xacro)
@@ -20,4 +20,9 @@
             <material name="black"/>
         </visual>
+        <collision>
+            <geometry>
+                <box size="0.001 0.001 0.001" />
+            </geometry>
+        </collision>
     </link>
     <joint name="camera_optical_joint" type="fixed">

File: src/articubot_one/description/face.xacro (robot description, xacro)
@@ -28,4 +28,9 @@
             <material name="red"/>
         </visual>
+        <collision>
+            <geometry>
+                <box size="0.001 0.001 0.001" />
+            </geometry>
+        </collision>
     </link>
     <gazebo reference="face_link">

Commit message: Added axles and moved camera

File: src/articubot_one/description/camera.xacro (robot description, xacro)
@@ -4,14 +4,14 @@
         <parent link="chassis"/>
         <child link="camera_link"/>
-        <origin xyz="0.23 0 0.081" rpy="0 0.18 0"/>
+        <origin xyz="0.255 0 0.04" rpy="0 0 0"/>
     </joint>
     <link name="camera_link">
         <visual>
             <geometry>
-                <box size="0.010 0.03 0.03"/>
+                <box size="0.010 0.05 0.025"/>
             </geometry>
             <material name="black"/>
         </visual>
-        <visual>
+        <!-- <visual>
             <origin xyz="0 0 -0.02"/>
             <geometry>
@@ -19,5 +19,5 @@
             </geometry>
             <material name="black"/>
-        </visual>
+        </visual> -->
         <collision>
             <geometry>

File: src/articubot_one/description/robot_core.xacro (robot description, xacro)
@@ -123,4 +123,11 @@
             <material name="blue"/>
         </visual>
+        <visual>
+            <origin xyz="0 0 ${-wheel_thickness/2}" rpy="0 0 0"/>
+            <geometry>
+                <cylinder radius="0.005" length="0.03"/>
+            </geometry>
+            <material name="blue"/>
+        </visual>
         <collision>
             <geometry>
@@ -146,4 +153,11 @@
             <geometry>
                 <cylinder radius="${wheel_radius}" length="${wheel_thickness}"/>
+            </geometry>
+            <material name="blue"/>
+        </visual>
+        <visual>
+            <origin xyz="0 0 ${-wheel_thickness/2}" rpy="0 0 0"/>
+            <geometry>
+                <cylinder radius="0.005" length="0.03"/>
             </geometry>
             <material name="blue"/>
