Commit message: Check xacro files

File: src/articubot_one/description/imu.xacro (robot description, xacro)
@@ -4,5 +4,5 @@
         <parent link="chassis" />
         <child link="imu_link" />
-        <origin xyz="0.235 0 0.15" rpy="0 0 0"/>
+        <origin xyz="0.235 0 0.14" rpy="0 0 0"/>
     </joint>
     <link name="imu_link">

File: src/articubot_one/description/robot.urdf.xacro (robot description, xacro)
@@ -13,8 +13,7 @@
     <xacro:include filename="camera.xacro" />
     <xacro:include filename="imu.xacro" />
+    <!-- <xacro:include filename="depth_camera.xacro" /> -->
+    <xacro:include filename="face.xacro" />
     <!-- <xacro:include filename="rrbot.urdf.xacro" /> -->
     <xacro:include filename="$(find robot_arm)/urdf/robot_arm.urdf" />
-    <!-- <xacro:include filename="robot_arm.xacro" />    -->
-    <!-- <xacro:include filename="depth_camera.xacro" /> -->
-    <!-- <xacro:include filename="face.xacro" />         -->
 </robot>

File: src/robot_arm/urdf/robot_arm.urdf (robot description, URDF)
Before this commit: robot robot_arm, 7 links, 7 joints
Links:
- link base_link_arm: mass 0.35184 -> 0.035184
- link link1: mass 0.17883 -> 0.017883
- link link2: mass 0.073669 -> 0.0073669
- link link3: mass 0.0853549537054368 -> 0.00853549537054368
- link link4: mass 0.0614391558855416 -> 0.00614391558855416
- link link51: mass 0.00475482638149408 -> 0.000475482638149408
- link link52: mass 0.00475475613653127 -> 0.000475475613653127
Joints:
- joint base_joint_arm: origin xyz=0.05 0 0.15 rpy=0 0 0 -> xyz=-0.15 0 0.13 rpy=0 0 0; parent chassis -> base_link

Commit message: Gazebo still not working

File: src/articubot_one/description/imu.xacro (robot description, xacro)
@@ -15,8 +15,8 @@
         <collision>
             <geometry>
-                <box size="0.1 0.1 0.1" />
+                <box size="0.05 0.05 0.05" />
             </geometry>
         </collision>
-        <xacro:inertial_box mass="0.1" x="0.1" y="0.1" z="0.1" >
+        <xacro:inertial_box mass="0.01" x="0.05" y="0.05" z="0.05" >
             <origin xyz="0 0 0"  rpy="0 0 0" />
         </xacro:inertial_box>

File: src/articubot_one/description/ros2_control.xacro (robot description, xacro)
@@ -99,5 +99,5 @@
                 <state_interface name="position" />
             </joint> -->
-            <joint name="joint2">
+            <joint name="joint4">
                 <command_interface name="position">
                     <param name="min">-1</param>

Commit message: Added raspi and adjusted imu + lidar

File: src/articubot_one/description/imu.xacro (robot description, xacro)
@@ -4,10 +4,10 @@
         <parent link="chassis" />
         <child link="imu_link" />
-        <origin xyz="0.08 0 0.045" rpy="0 0 0"/>
+        <origin xyz="0.02 0.02 0.11" rpy="0 0 0"/>
     </joint>
     <link name="imu_link">
         <visual>
             <geometry>
-                <box size="0.03 0.03 0.015" />
+                <box size="0.02 0.01 0.004" />
             </geometry>
             <material name="red"/>

File: src/articubot_one/description/lidar.xacro (robot description, xacro)
@@ -4,10 +4,10 @@
         <parent link="chassis"/>
         <child link="laser_frame"/>
-        <origin xyz="0.025 0 0.10" rpy="0 0 0"/>
+        <origin xyz="0.075 0 0.14" rpy="0 0 0"/>
     </joint>
     <link name="laser_frame">
         <visual>
             <geometry>
-                <cylinder radius="0.05" length="0.04"/>
+                <cylinder radius="0.05" length="0.03"/>
             </geometry>
             <material name="yellow"/>
@@ -22,5 +22,5 @@
         <collision>
             <geometry>
-                <cylinder radius="0.05" length="0.04"/>
+                <cylinder radius="0.05" length="0.03"/>
             </geometry>
         </collision>

File: src/articubot_one/description/robot_core.xacro (robot description, xacro)
@@ -3,5 +3,5 @@
     <xacro:include filename="inertial_macros.xacro"/>
     <xacro:property name="chassis_length" value="0.25"/>    <!-- 335"/>     -->
-    <xacro:property name="chassis_width" value="0.125"/>    <!-- 265"/>     -->
+    <xacro:property name="chassis_width" value="0.130"/>    <!-- 265"/>     -->
     <xacro:property name="chassis_height" value="0.04"/>   <!-- 138"/>     -->
     <!-- <xacro:property name="chassis_extension_length" value="0.15"/>
@@ -202,3 +202,30 @@
         <mu2 value="0.001"/>
     </gazebo>
+    <!-- RaspPi4 -->
+    <joint name="raspi_joint" type="fixed">
+        <parent link="chassis"/>
+        <child link="raspi"/>
+        <origin xyz="0.01 -0.03 0.04" rpy="0 -${pi/2} 0"/>
+    </joint>
+    <link name="raspi">
+        <visual>
+            <origin xyz="0.04 0.03 0.005"/>
+            <geometry>
+                <box size="0.08 0.06 0.01"/>
+            </geometry>
+            <material name="orange"/>
+        </visual>
+        <collision>
+            <origin xyz="0.04 0.03 0.005"/>
+            <geometry>
+                <box size="0.08 0.06 0.01"/>
+            </geometry>
+        </collision>
+        <xacro:inertial_box mass="0.05" x="0.08" y="0.06" z="0.01">
+            <origin xyz="0.04 0.03 0.005" rpy="0 0 0"/>
+        </xacro:inertial_box>
+    </link>
+    <gazebo reference="raspi">
+        <material>Gazebo/Orange</material>
+    </gazebo>
 </robot>
