Commit message: Move arm to top of chassis

File: src/robot_arm/urdf/robot_arm.urdf (robot description, URDF)
Before this commit: robot robot_arm, 7 links, 7 joints
Joints:
- joint base_joint_arm: origin  -> xyz=0.05 0 0.15 rpy=0 0 0; parent base_link -> chassis

Commit message: Works for both gazebo + rviz2

File: src/robot_arm/urdf/robot_arm.urdf (robot description, URDF)
Before this commit: robot robot_arm, 7 links, 7 joints
Links:
- link base_link_arm: geometry collision mesh filename=file://$(find robot_arm)/meshes/base_link.STL; visual mesh filename=file://$(find robot_arm)/meshes/base_link.STL
- link link1: geometry collision mesh filename=file://$(find robot_arm)/meshes/link1.STL; visual mesh filename=file://$(find robot_arm)/meshes/link1.STL
- link link2: geometry collision mesh filename=file://$(find robot_arm)/meshes/link2.STL; visual mesh filename=file://$(find robot_arm)/meshes/link2.STL
- link link3: geometry collision mesh filename=file://$(find robot_arm)/meshes/link3.STL; visual mesh filename=file://$(find robot_arm)/meshes/link3.STL
- link link4: geometry collision mesh filename=file://$(find robot_arm)/meshes/link4.STL; visual mesh filename=file://$(find robot_arm)/meshes/link4.STL
- link link51: geometry collision mesh filename=file://$(find robot_arm)/meshes/link51.STL; visual mesh filename=file://$(find robot_arm)/meshes/link51.STL
- link link52: geometry collision mesh filename=file://$(find robot_arm)/meshes/link52.STL; visual mesh filename=file://$(find robot_arm)/meshes/link52.STL
