Commit message: Eezybotarm visible on chasis

File: src/eezybotarm/urdf/eezybotarm.urdf (robot description, URDF)
Before this commit: robot eezybotarm, 9 links, 9 joints
Joints:
- joint base_joint_eezybotarm: origin xyz=-0.14 0 0.13 rpy=0 0 0 -> xyz=-0.12 -0.09 0.13 rpy=0 0 0

File: src/robot_arm/urdf/robot_arm.urdf (robot description, URDF)
Before this commit: robot robot_arm, 7 links, 7 joints
Joints:
- joint base_joint_arm: origin xyz=-0.14 0 0.13 rpy=0 0 0 -> xyz=-0.14 0.045 0.13 rpy=0 0 0
