Commit message: Renamed joint2v to joint_2v

File: src/eezybotarm/urdf/eezybotarm.urdf.xacro (robot description, xacro)
@@ -93,5 +93,5 @@
   </link>
   <!-- VIRTUAL MIMIC JOINT 2-->
-  <joint name="joint2v" type="revolute">
+  <joint name="joint_2v" type="revolute">
     <origin xyz="-0.021 0.135 -0.0105" rpy="1.570796325 0 0" />
     <parent link="link_2"/>

Commit message: Eezybotarm is stable but link_3 drops

File: src/eezybotarm/urdf/eezybotarm.urdf.xacro (robot description, xacro)
@@ -25,5 +25,5 @@
       <origin rpy="0 0 0" xyz="0 0 0"/>
     </collision>
-    <xacro:inertial_box mass="0.01" x="0.1" y="0.1" z="0.1">
+    <xacro:inertial_box mass="0.1" x="0.1" y="0.1" z="0.1">
       <origin xyz="0 0 0" rpy="0 0 0"/>
     </xacro:inertial_box>
@@ -58,5 +58,5 @@
       </geometry>
     </collision>
-    <xacro:inertial_box mass="0.001" x="0.01" y="0.01" z="0.01">
+    <xacro:inertial_box mass="0.05" x="0.1" y="0.1" z="0.1">
       <origin xyz="0 0 0" rpy="0 0 0"/>
     </xacro:inertial_box>
@@ -88,5 +88,5 @@
       </geometry>
     </collision>
-    <xacro:inertial_box mass="0.001" x="0.1" y="0.1" z="0.1">
+    <xacro:inertial_box mass="0.04" x="0.1" y="0.1" z="0.1">
       <origin xyz="0 0 0" rpy="0 0 0"/>
     </xacro:inertial_box>
@@ -129,4 +129,5 @@
     <limit effort="0" velocity="0"
       lower="-0.77" upper="0.45"/>
+    <dynamics damping="10.0" friction="10.0" />
   </joint>
 <!-- LINK 3 ELBOW -->
@@ -147,5 +148,5 @@
       </geometry>
     </collision>
-    <xacro:inertial_box mass="0.001" x="0.1" y="0.1" z="0.1">
+    <xacro:inertial_box mass="0.01" x="0.1" y="0.1" z="0.1">
       <origin xyz="0 0 0" rpy="0 0 0"/>
     </xacro:inertial_box>
