Commit message: rviz didn't like "spaces" in filenames

File: src/arduino_arm/urdf/arduino_arm_rviz2.urdf (robot description, URDF)
Before this commit: robot arduino_arm, 7 links, 7 joints
Links:
- added link base_link
Joints:
- joint base_joint_arduino_arm: origin xyz=-0.14 0 0.145 rpy=0 0 0 -> xyz=0 0 0 rpy=0 0 0
