Commit message: arduino_arm connected to forward_publisher

File: src/arduino_arm/urdf/arduino_arm.urdf.xacro (robot description, xacro)
@@ -1,5 +1,7 @@
 <?xml version="1.0"?>
+<robot xmlns:xacro="http://www.ros.org/wiki/xacro"  name="arduino_arm">
+<!-- <?xml version="1.0"?> -->
 <!-- created with Phobos 1.0.1 "Capricious Choutengan" -->
-<robot name="arduino_arm">
+<!-- <robot name="arduino_arm"> -->
 <!--
     <link name="base_link"/>
@@ -7,8 +9,8 @@
     <joint name="base_joint_arduino_arm" type="fixed">
         <parent link="base_link" />
-        <child link="base_arduino_arm" />
+        <child link="base_link_arduino_arm" />
         <origin xyz="-0.14 0 0.145" rpy="0 0 0" />
     </joint>
-    <link name="base_arduino_arm">
+    <link name="base_link_arduino_arm">
         <inertial>
             <origin xyz="0 0 0" rpy="0 0 0" />
@@ -33,5 +35,5 @@
         </collision>
     </link>
-    <link name="waist">
+    <link name="waist_link">
         <inertial>
             <origin xyz="0 0 0" rpy="0 0 0" />
@@ -176,6 +178,6 @@
     <joint name="base_joint" type="revolute">
         <origin xyz="-0.00345 -1e-05 0.04449" rpy="0 0 0" />
-        <parent link="base_arduino_arm" />
-        <child link="waist" />
+        <parent link="base_link_arduino_arm" />
+        <child link="waist_link" />
         <axis xyz="0 0 1.0" />
         <limit lower="-1.571" upper="1.571" effort="1000.0" velocity="1.0" />
@@ -183,5 +185,5 @@
     <joint name="shoulder" type="revolute">
         <origin xyz="0.00396 0.01369 0.03521" rpy="1.5708 0.03778 1.5708" />
-        <parent link="waist" />
+        <parent link="waist_link" />
         <child link="arm1" />
         <axis xyz="0 0 1.0" />
@@ -282,8 +284,8 @@
         </plugin>
     </gazebo>
-    <gazebo reference="base_arduino_arm">
+    <gazebo reference="base_link_arduino_arm">
         <material>Gazebo/Green</material>
     </gazebo>
-    <gazebo reference="waist">
+    <gazebo reference="waist_link">
         <material>Gazebo/Green</material>
     </gazebo>

File: src/articubot_one/description/imu.xacro (robot description, xacro)
@@ -4,5 +4,5 @@
         <parent link="chassis" />
         <child link="imu_link" />
-        <origin xyz="0.28 0 0.14" rpy="0 0 0"/>
+        <origin xyz="0.26 0 0.14" rpy="0 0 0"/>
     </joint>
     <link name="imu_link">

File: src/articubot_one/description/lidar.xacro (robot description, xacro)
@@ -4,5 +4,5 @@
         <parent link="chassis"/>
         <child link="laser_frame"/>
-        <origin xyz="0.235 0 0.212" rpy="0 0 0"/>
+        <origin xyz="0.20 0 0.212" rpy="0 0 0"/>
     </joint>
     <link name="laser_frame">

File: src/articubot_one/description/robot.urdf.xacro (robot description, xacro)
@@ -18,4 +18,4 @@
     <!-- <xacro:include filename="$(find robot_arm)/urdf/robot_arm.urdf" /> -->
     <!-- <xacro:include filename="$(find eezybotarm)/urdf/eezybotarm.urdf.xacro" /> -->
-    <xacro:include filename="$(find arduino_arm)/urdf/arduino_arm.urdf" />
+    <xacro:include filename="$(find arduino_arm)/urdf/arduino_arm.urdf.xacro" />
 </robot>

File: src/articubot_one/description/ros2_control.xacro (robot description, xacro)
@@ -42,32 +42,4 @@
             </joint>
         </ros2_control>
-        <!-- <ros2_control name="RealRobot" type="system">
-            <hardware>
-                <plugin>diffdrive_arduino/DiffDriveArduino</plugin>
-                <param name="left_wheel_name">left_wheel_joint</param>
-                <param name="right_wheel_name">right_wheel_joint</param>
-                <param name="loop_rate">30</param>
-                <param name="device">/dev/ttyUSB0</param>
-                <param name="baud_rate">57600</param>
-                <param name="timeout">1000</param>
-                <param name="enc_counts_per_rev">3436</param>
-            </hardware>
-            <joint name="left_wheel_joint">
-                <command_interface name="velocity">
-                    <param name="min">-10</param>
-                    <param name="max">10</param>
-                </command_interface>
-                <state_interface name="velocity" />
-                <state_interface name="position" />
-            </joint>
-            <joint name="right_wheel_joint">
-                <command_interface name="velocity">
-                    <param name="min">-10</param>
-                    <param name="max">10</param>
-                </command_interface>
-                <state_interface name="velocity" />
-                <state_interface name="position" />
-            </joint>
-        </ros2_control> -->
     </xacro:unless>
     <xacro:if value="$(arg sim_mode)">
@@ -92,5 +64,5 @@
                 <state_interface name="position" />
             </joint>
-            <joint name="joint1">
+            <joint name="base_joint">
                 <command_interface name="position">
                     <param name="min">-1</param>
@@ -99,5 +71,5 @@
                 <state_interface name="position" />
             </joint>
-            <joint name="joint2">
+            <joint name="shoulder">
                 <command_interface name="position">
                     <param name="min">-1</param>
@@ -106,5 +78,5 @@
                 <state_interface name="position" />
             </joint>
-            <joint name="joint3">
+            <joint name="elbow">
                 <command_interface name="position">
                     <param name="min">-1</param>
@@ -113,62 +85,6 @@
                 <state_interface name="position" />
             </joint>
-            <joint name="joint4">
-                <command_interface name="position">
-                    <param name="min">-1</param>
-                    <param name="max">1</param>
-                </command_interface>
-                <state_interface name="position" />
-            </joint>
-            <joint name="joint51">
-                <command_interface name="position">
-                    <param name="min">-1</param>
-                    <param name="max">1</param>
-                </command_interface>
-                <state_interface name="position" />
-            </joint>
-            <joint name="joint52">
-                <command_interface name="position">
-                    <param name="min">-1</param>
-                    <param name="max">1</param>
-                </command_interface>
-                <state_interface name="position" />
-            </joint>
-        <joint name="joint_1">
-            <command_interface name="position">
-                <param name="min">-1</param>
-                <param name="max">1</param>
-            </command_interface>
-            <state_interface name="position" />
-        </joint>
-        <joint name="joint_2">
-            <command_interface name="position">
-                <param name="min">-1</param>
-                <param name="max">1</param>
-            </command_interface>
-            <state_interface name="position" />
-        </joint>
-        <joint name="joint_2v">
-            <command_interface name="position">
-                <param name="min">-1</param>
-                <param name="max">1</param>
-            </command_interface>
-            <state_interface name="position" />
-        </joint>
-        <joint name="joint_3">
-            <command_interface name="position">
-                <param name="min">-1</param>
-                <param name="max">1</param>
-            </command_interface>
-            <state_interface name="position" />
-        </joint>
-        <joint name="joint_4">
-            <command_interface name="position">
-                <param name="min">-1</param>
-                <param name="max">1</param>
-            </command_interface>
-            <state_interface name="position" />
-        </joint>
-    </ros2_control>
-</xacro:if>
+        </ros2_control>
+    </xacro:if>
     <gazebo>
         <plugin name="gazebo_ros2_control" filename="libgazebo_ros2_control.so">

Commit message: Some issues with colors in gaz + rviz

File: src/arduino_arm/urdf/arduino_arm.urdf.xacro (robot description, xacro)
@@ -4,7 +4,5 @@
 <!-- created with Phobos 1.0.1 "Capricious Choutengan" -->
 <!-- <robot name="arduino_arm"> -->
-<!--
-    <link name="base_link"/>
--->
+<!-- <link name="base_link"/> -->
     <joint name="base_joint_arduino_arm" type="fixed">
         <parent link="base_link" />
@@ -59,5 +57,5 @@
         </collision>
     </link>
-    <link name="arm1">
+    <link name="arm1_link">
         <inertial>
             <origin xyz="0 0 0" rpy="0 0 0" />
@@ -82,5 +80,5 @@
         </collision>
     </link>
-    <link name="arm2">
+    <link name="arm2_link">
         <inertial>
             <origin xyz="0 0 0" rpy="0 0 0" />
@@ -105,5 +103,5 @@
         </collision>
     </link>
-    <link name="arm3">
+    <link name="arm3_link">
         <inertial>
             <origin xyz="0 0 0" rpy="0 0 0" />
@@ -129,5 +127,5 @@
         </collision>
     </link>
-    <link name="gripper1">
+    <link name="gripper1_link">
         <inertial>
             <origin xyz="0 0 0" rpy="0 0 0" />
@@ -142,5 +140,5 @@
             </geometry>
             <material name="">
-                <color rgba="0 1 0 1" />
+                <color rgba="0.7 1 0 1" />
             </material>
         </visual>
@@ -153,5 +151,5 @@
         </collision>
     </link>
-    <link name="gripper2">
+    <link name="gripper2_link">
         <inertial>
             <origin xyz="0 0 0" rpy="0 0 0" />
@@ -165,5 +163,5 @@
             </geometry>
             <material name="">
-                <color rgba="0 1 0 1" />
+                <color rgba="0.7 1 0 1" />
             </material>
         </visual>
@@ -176,5 +174,5 @@
         </collision>
     </link>
-    <joint name="base_joint" type="revolute">
+    <joint name="base_arduino_arm_joint" type="revolute">
         <origin xyz="-0.00345 -1e-05 0.04449" rpy="0 0 0" />
         <parent link="base_link_arduino_arm" />
@@ -183,39 +181,39 @@
         <limit lower="-1.571" upper="1.571" effort="1000.0" velocity="1.0" />
     </joint>
-    <joint name="shoulder" type="revolute">
+    <joint name="shoulder_joint" type="revolute">
         <origin xyz="0.00396 0.01369 0.03521" rpy="1.5708 0.03778 1.5708" />
         <parent link="waist_link" />
-        <child link="arm1" />
+        <child link="arm1_link" />
         <axis xyz="0 0 1.0" />
         <limit lower="-1.571" upper="1.571" effort="1000.0" velocity="1.0" />
     </joint>
-    <joint name="elbow" type="revolute">
+    <joint name="elbow_joint" type="revolute">
         <origin xyz="-7e-05 0.11689 -0.00792" rpy="-0.0013 -3.14159 0.03778" />
-        <parent link="arm1" />
-        <child link="arm2" />
+        <parent link="arm1_link" />
+        <child link="arm2_link" />
         <axis xyz="0 0 1.0" />
         <limit lower="-1.57" upper="1.57" effort="1000.0" velocity="1.0" />
     </joint>
-    <joint name="wrist" type="revolute">
+    <joint name="wrist_joint" type="revolute">
         <origin xyz="-0.0088 0.12752 -0.00487" rpy="-0.01458 3.14159 0" />
-        <parent link="arm2" />
-        <child link="arm3" />
+        <parent link="arm2_link" />
+        <child link="arm3_link" />
         <axis xyz="0 0 1.0" />
         <limit lower="-1.57" upper="1.57" effort="1000.0" velocity="1.0" />
     </joint>
-    <joint name="gripper" type="revolute">
+    <joint name="gripper1_joint" type="revolute">
         <origin xyz="-0.02735 0.03009 -0.02013" rpy="-1.27431 -1.58408 1.5708" />
-        <parent link="arm3" />
-        <child link="gripper1" />
+        <parent link="arm3_link" />
+        <child link="gripper1_link" />
         <axis xyz="0 0 1.0" />
         <limit lower="0" upper="1.047" effort="1000.0" velocity="1.0" />
     </joint>
-    <joint name="gripper22" type="revolute">
+    <joint name="gripper2_joint" type="revolute">
         <origin xyz="-0.02492 0.03048 0.00564" rpy="-1.25673 -1.55752 -1.57079" />
-        <parent link="arm3" />
-        <child link="gripper2" />
+        <parent link="arm3_link" />
+        <child link="gripper2_link" />
         <axis xyz="0 0 1.0" />
         <limit lower="0" upper="1.047" effort="1000.0" velocity="1.0" />
-        <mimic joint="gripper" multiplier="1.0" offset="0.0" />
+        <!-- <mimic joint="gripper1_joint" multiplier="1.0" offset="0.0" /> -->
     </joint>
     <transmission name="trans_base_joint">
@@ -231,5 +229,5 @@
     <transmission name="trans_shoulder">
         <type>transmission_interface/SimpleTransmission</type>
-        <joint name="shoulder">
+        <joint name="shoulder_joint">
             <hardwareInterface>hardware_interface/PositionJointInterface</hardwareInterface>
         </joint>
@@ -241,5 +239,5 @@
     <transmission name="trans_elbow">
         <type>transmission_interface/SimpleTransmission</type>
-        <joint name="elbow">
+        <joint name="elbow_joint">
             <hardwareInterface>hardware_interface/PositionJointInterface</hardwareInterface>
         </joint>
@@ -251,5 +249,5 @@
     <transmission name="trans_wrist">
         <type>transmission_interface/SimpleTransmission</type>
-        <joint name="wrist">
+        <joint name="wrist_joint">
             <hardwareInterface>hardware_interface/PositionJointInterface</hardwareInterface>
         </joint>
@@ -261,5 +259,5 @@
     <transmission name="trans_gripper">
         <type>transmission_interface/SimpleTransmission</type>
-        <joint name="gripper">
+        <joint name="gripper1_joint">
             <hardwareInterface>hardware_interface/PositionJointInterface</hardwareInterface>
         </joint>
@@ -271,5 +269,5 @@
     <transmission name="trans_gripper2">
         <type>transmission_interface/SimpleTransmission</type>
-        <joint name="gripper2">
+        <joint name="gripper2_joint">
             <hardwareInterface>hardware_interface/EffortJointInterface</hardwareInterface>
         </joint>

File: src/articubot_one/description/ros2_control.xacro (robot description, xacro)
@@ -64,5 +64,5 @@
                 <state_interface name="position" />
             </joint>
-            <joint name="base_joint">
+            <joint name="base_arduino_arm_joint">
                 <command_interface name="position">
                     <param name="min">-1</param>
@@ -71,5 +71,5 @@
                 <state_interface name="position" />
             </joint>
-            <joint name="shoulder">
+            <joint name="shoulder_joint">
                 <command_interface name="position">
                     <param name="min">-1</param>
@@ -78,5 +78,26 @@
                 <state_interface name="position" />
             </joint>
-            <joint name="elbow">
+            <joint name="elbow_joint">
+                <command_interface name="position">
+                    <param name="min">-1</param>
+                    <param name="max">1</param>
+                </command_interface>
+                <state_interface name="position" />
+            </joint>
+            <joint name="wrist_joint">
+                <command_interface name="position">
+                    <param name="min">-1</param>
+                    <param name="max">1</param>
+                </command_interface>
+                <state_interface name="position" />
+            </joint>
+            <joint name="gripper1_joint">
+                <command_interface name="position">
+                    <param name="min">-1</param>
+                    <param name="max">1</param>
+                </command_interface>
+                <state_interface name="position" />
+            </joint>
+            <joint name="gripper2_joint">
                 <command_interface name="position">
                     <param name="min">-1</param>

Commit message: Patched the gripper stl files

File: src/arduino_arm/urdf/arduino_arm.urdf.xacro (robot description, xacro)
@@ -134,18 +134,18 @@
         </inertial>
         <visual name="Gripper1">
-            <origin xyz="0 0 0" rpy="-1.86728 0 0" />
-            <geometry>
-                <mesh filename="file://$(find arduino_arm)/meshes/Gripper1.002.stl"
-                    scale="1.0 1.0 1.0" />
-            </geometry>
-            <material name="">
-                <color rgba="0.7 1 0 1" />
+            <origin xyz="0 -0.01 0.014" rpy="-1.86728 0 0" />
+            <geometry>
+                <mesh filename="file://$(find arduino_arm)/meshes/gripper1_fix.stl"
+                    scale="0.001 0.001 0.001" />
+            </geometry>
+            <material name="">
+                <color rgba="0 1 1 1" />
             </material>
         </visual>
         <collision name="Gripper1.000">
-            <origin xyz="0.00072 0.00044 0.00014" rpy="-1.86728 0 0" />
-            <geometry>
-                <mesh filename="file://$(find arduino_arm)/meshes/Gripper1.003.stl"
-                    scale="1.0 1.0 1.0" />
+            <origin xyz="0 -0.01 0.014" rpy="-1.86728 0 0" />
+            <geometry>
+                <mesh filename="file://$(find arduino_arm)/meshes/gripper1_fix.stl"
+                    scale="0.001 0.001 0.001" />
             </geometry>
         </collision>
@@ -158,17 +158,17 @@
         </inertial>
         <visual name="Gripper2">
-            <origin xyz="0 0 0" rpy="1.25673 0 0" />
-            <geometry>
-                <mesh filename="file://$(find arduino_arm)/meshes/Gripper2.stl" scale="1.0 1.0 1.0" />
-            </geometry>
-            <material name="">
-                <color rgba="0.7 1 0 1" />
+            <origin xyz="-0.0015 0.01 -0.014" rpy="1.25673 0 0" />
+            <geometry>
+                <mesh filename="file://$(find arduino_arm)/meshes/gripper2_fix.stl" scale="0.001 0.001 0.001" />
+            </geometry>
+            <material name="">
+                <color rgba="0 1 1 1" />
             </material>
         </visual>
         <collision name="Gripper2.000">
-            <origin xyz="-0.00023 -0.00045 0.00034" rpy="1.25673 0 0" />
-            <geometry>
-                <mesh filename="file://$(find arduino_arm)/meshes/Gripper2.001.stl"
-                    scale="1.0 1.0 1.0" />
+            <origin xyz="-0.0015 0.01 -0.014" rpy="1.25673 0 0" />
+            <geometry>
+                <mesh filename="file://$(find arduino_arm)/meshes/gripper2_fix.stl"
+                    scale="0.001 0.001 0.001" />
             </geometry>
         </collision>
@@ -278,10 +278,7 @@
     </transmission>
     <gazebo>
-        <plugin name="gazebo_ros_control" filename="libgazebo_ros_control.so">
+        <plugin name="gazebo_ros2_control" filename="libgazebo_ros_control.so">
             <robotNamespace>/</robotNamespace>
         </plugin>
-    </gazebo>
-    <gazebo reference="base_link_arduino_arm">
-        <material>Gazebo/Green</material>
     </gazebo>
     <gazebo reference="waist_link">

Commit message: All works except arduino_arm gazebo colours

File: src/arduino_arm/urdf/arduino_arm.urdf.xacro (robot description, xacro)
@@ -158,5 +158,5 @@
         </inertial>
         <visual name="Gripper2">
-            <origin xyz="-0.0015 0.01 -0.014" rpy="1.25673 0 0" />
+            <origin xyz="-0.0015 0.01 -0.0165" rpy="1.25673 0 0" />
             <geometry>
                 <mesh filename="file://$(find arduino_arm)/meshes/gripper2_fix.stl" scale="0.001 0.001 0.001" />
@@ -167,11 +167,11 @@
         </visual>
         <collision name="Gripper2.000">
-            <origin xyz="-0.0015 0.01 -0.014" rpy="1.25673 0 0" />
-            <geometry>
-                <mesh filename="file://$(find arduino_arm)/meshes/gripper2_fix.stl"
-                    scale="0.001 0.001 0.001" />
-            </geometry>
-        </collision>
-    </link>
+            <origin xyz="-0.0015 0.01 -0.0165" rpy="1.25673 0 0" />
+            <geometry>
+	    	<cylinder length="0.001" radius="0.001"/>
+            </geometry>
+        </collision>
+    </link>
+		    <!--                <mesh filename="file://$(find arduino_arm)/meshes/gripper2_fix.stl" scale="0.001 0.001 0.001" /> -->
     <joint name="base_arduino_arm_joint" type="revolute">
         <origin xyz="-0.00345 -1e-05 0.04449" rpy="0 0 0" />
@@ -215,5 +215,5 @@
         <axis xyz="0 0 1.0" />
         <limit lower="0" upper="1.047" effort="1000.0" velocity="1.0" />
-        <!-- <mimic joint="gripper1_joint" multiplier="1.0" offset="0.0" /> -->
+	<mimic joint="gripper1_joint" multiplier="1.0" offset="0.0" />
     </joint>
     <transmission name="trans_base_joint">
@@ -267,4 +267,5 @@
         </actuator>
     </transmission>
+    <!--
     <transmission name="trans_gripper2">
         <type>transmission_interface/SimpleTransmission</type>
@@ -277,4 +278,5 @@
         </actuator>
     </transmission>
+    -->
     <gazebo>
         <plugin name="gazebo_ros2_control" filename="libgazebo_ros_control.so">
