Commit message: Remove robot_arm & eezybotarm

File: src/arduino_arm/urdf/arduino_arm.urdf.xacro (robot description, xacro)
@@ -16,5 +16,5 @@
             <inertia ixx="0.001" ixy="0" ixz="0" iyy="0.001" iyz="0" izz="0.001" />
         </inertial>
-        <visual name="Base">
+        <visual>
             <origin xyz="0 0 0" rpy="1.5708 0 0" />
             <geometry>
@@ -26,5 +26,5 @@
             </material>
         </visual>
-        <collision name="Base">
+        <collision>
             <origin xyz="-0.0029 0.00016 0.01165" rpy="3.14159 0 0" />
             <geometry>
@@ -39,5 +39,5 @@
             <inertia ixx="0.001" ixy="0" ixz="0" iyy="0.001" iyz="0" izz="0.001" />
         </inertial>
-        <visual name="Waist">
+        <visual>
             <origin xyz="0 0 0" rpy="1.5708 0 0" />
             <geometry>
@@ -49,5 +49,5 @@
             </material>
         </visual>
-        <collision name="Waist.000">
+        <collision>
             <origin xyz="0.00019 0 3e-05" rpy="1.5708 0 0" />
             <geometry>
@@ -63,5 +63,5 @@
             <inertia ixx="0.001" ixy="0" ixz="0" iyy="0.001" iyz="0" izz="0.001" />
         </inertial>
-        <visual name="Arm_01">
+        <visual>
             <origin xyz="0 0 0" rpy="0 0 0" />
             <geometry>
@@ -73,5 +73,5 @@
             </material>
         </visual>
-        <collision name="Arm_01">
+        <collision>
             <origin xyz="-0.00032 0.05624 0.00439" rpy="0 0 0" />
             <geometry>
@@ -86,5 +86,5 @@
             <inertia ixx="0.001" ixy="0" ixz="0" iyy="0.001" iyz="0" izz="0.001" />
         </inertial>
-        <visual name="Arm_02">
+        <visual>
             <origin xyz="0 0 0" rpy="-1.48894 -1.57209 1.57067" />
             <geometry>
@@ -96,5 +96,5 @@
             </material>
         </visual>
-        <collision name="Arm_02">
+        <collision>
             <origin xyz="-0.00436 0.05688 0.00738" rpy="-1.48879 -1.57209 1.57066" />
             <geometry>
@@ -109,5 +109,5 @@
             <inertia ixx="0.001" ixy="0" ixz="0" iyy="0.001" iyz="0" izz="0.001" />
         </inertial>
-        <visual name="Arm_03">
+        <visual>
             <origin xyz="0 0 0" rpy="1.2416 1.55752 1.5708" />
             <geometry>
@@ -119,5 +119,5 @@
             </material>
         </visual>
-        <collision name="Arm_03.000">
+        <collision>
             <origin xyz="-0.00062 0.00019 0.00049" rpy="1.24161 1.55752 1.5708" />
             <geometry>
@@ -133,5 +133,5 @@
             <inertia ixx="0.001" ixy="0" ixz="0" iyy="0.001" iyz="0" izz="0.001" />
         </inertial>
-        <visual name="Gripper1">
+        <visual>
             <origin xyz="0 -0.01 0.014" rpy="-1.86728 0 0" />
             <geometry>
@@ -143,5 +143,5 @@
             </material>
         </visual>
-        <collision name="Gripper1.000">
+        <collision>
             <origin xyz="0 -0.01 0.014" rpy="-1.86728 0 0" />
             <geometry>
@@ -157,5 +157,5 @@
             <inertia ixx="0.001" ixy="0" ixz="0" iyy="0.001" iyz="0" izz="0.001" />
         </inertial>
-        <visual name="Gripper2">
+        <visual>
             <origin xyz="-0.0015 0.01 -0.0165" rpy="1.25673 0 0" />
             <geometry>
@@ -166,5 +166,5 @@
             </material>
         </visual>
-        <collision name="Gripper2.000">
+        <collision>
             <origin xyz="-0.0015 0.01 -0.0165" rpy="1.25673 0 0" />
             <geometry>
@@ -173,5 +173,4 @@
         </collision>
     </link>
-		    <!--                <mesh filename="file://$(find arduino_arm)/meshes/gripper2_fix.stl" scale="0.001 0.001 0.001" /> -->
     <joint name="base_arduino_arm_joint" type="revolute">
         <origin xyz="-0.00345 -1e-05 0.04449" rpy="0 0 0" />
@@ -284,6 +283,24 @@
         </plugin>
     </gazebo>
+    <gazebo reference="base_link_arduino_arm">
+        <material>Gazebo/Green</material>
+    </gazebo>
     <gazebo reference="waist_link">
         <material>Gazebo/Green</material>
     </gazebo>
+    <gazebo reference="arm1_link">
+        <material>Gazebo/Green</material>
+    </gazebo>
+    <gazebo reference="arm2_link">
+        <material>Gazebo/Green</material>
+    </gazebo>
+    <gazebo reference="arm3_link">
+        <material>Gazebo/Green</material>
+    </gazebo>
+    <gazebo reference="gripper1_link">
+        <material>Gazebo/Green</material>
+    </gazebo>
+    <gazebo reference="gripper2_link">
+        <material>Gazebo/Green</material>
+    </gazebo>
 </robot>

File: src/arduino_arm/urdf/arduino_arm_moveit.urdf.xacro (robot description, xacro)
@@ -159,5 +159,5 @@
             <inertia ixx="0.001" ixy="0" ixz="0" iyy="0.001" iyz="0" izz="0.001" />
         </inertial>
-        <visual name="Gripper2">
+        <visual>
             <origin xyz="-0.0015 0.01 -0.0165" rpy="1.25673 0 0" />
             <geometry>
@@ -168,5 +168,5 @@
             </material>
         </visual>
-        <collision name="Gripper2.000">
+        <collision>
             <origin xyz="-0.0015 0.01 -0.0165" rpy="1.25673 0 0" />
             <geometry>
@@ -175,5 +175,4 @@
         </collision>
     </link>
-		    <!--                <mesh filename="file://$(find arduino_arm)/meshes/gripper2_fix.stl" scale="0.001 0.001 0.001" /> -->
     <joint name="base_arduino_arm_joint" type="revolute">
         <origin xyz="-0.00345 -1e-05 0.04449" rpy="0 0 0" />
@@ -286,6 +285,9 @@
         </plugin>
     </gazebo>
-    <gazebo reference="waist_link">
-        <material>Gazebo/Green</material>
+    <gazebo reference="gripper2_link">
+    	<material>Gazebo/Green</material>
+	<visual>
+            <transparency>0.25</transparency>
+        </visual>
     </gazebo>
 </robot>

Commit message: Trying moveit with mobile robot

File: src/arduino_arm/urdf/arduino_arm.urdf.xacro (robot description, xacro)
@@ -5,5 +5,5 @@
 <!-- <robot name="arduino_arm"> -->
 <!-- <link name="base_link"/> -->
-    <joint name="base_joint_arduino_arm" type="fixed">
+    <joint name="base_link_arduino_arm_joint" type="fixed">
         <parent link="base_link" />
         <child link="base_link_arduino_arm" />
@@ -173,5 +173,5 @@
         </collision>
     </link>
-    <joint name="base_arduino_arm_joint" type="revolute">
+    <joint name="base_waist_joint" type="revolute">
         <origin xyz="-0.00345 -1e-05 0.04449" rpy="0 0 0" />
         <parent link="base_link_arduino_arm" />

File: src/arduino_arm/urdf/arduino_arm_moveit.urdf.xacro (robot description, xacro)
@@ -4,12 +4,10 @@
 <!-- created with Phobos 1.0.1 "Capricious Choutengan" -->
 <!-- <robot name="arduino_arm"> -->
-<!-- <link name="base_link"/> -->
-<!--
-    <joint name="base_joint_arduino_arm" type="fixed">
+    <link name="base_link"/>
+    <joint name="base_link_arduino_arm_joint" type="fixed">
         <parent link="base_link" />
         <child link="base_link_arduino_arm" />
         <origin xyz="-0.14 0 0.145" rpy="0 0 0" />
     </joint>
--->
     <link name="base_link_arduino_arm">
         <inertial>
@@ -18,5 +16,5 @@
             <inertia ixx="0.001" ixy="0" ixz="0" iyy="0.001" iyz="0" izz="0.001" />
         </inertial>
-        <visual name="Base">
+        <visual>
             <origin xyz="0 0 0" rpy="1.5708 0 0" />
             <geometry>
@@ -28,5 +26,5 @@
             </material>
         </visual>
-        <collision name="Base">
+        <collision>
             <origin xyz="-0.0029 0.00016 0.01165" rpy="3.14159 0 0" />
             <geometry>
@@ -41,5 +39,5 @@
             <inertia ixx="0.001" ixy="0" ixz="0" iyy="0.001" iyz="0" izz="0.001" />
         </inertial>
-        <visual name="Waist">
+        <visual>
             <origin xyz="0 0 0" rpy="1.5708 0 0" />
             <geometry>
@@ -51,5 +49,5 @@
             </material>
         </visual>
-        <collision name="Waist.000">
+        <collision>
             <origin xyz="0.00019 0 3e-05" rpy="1.5708 0 0" />
             <geometry>
@@ -65,5 +63,5 @@
             <inertia ixx="0.001" ixy="0" ixz="0" iyy="0.001" iyz="0" izz="0.001" />
         </inertial>
-        <visual name="Arm_01">
+        <visual>
             <origin xyz="0 0 0" rpy="0 0 0" />
             <geometry>
@@ -75,5 +73,5 @@
             </material>
         </visual>
-        <collision name="Arm_01">
+        <collision>
             <origin xyz="-0.00032 0.05624 0.00439" rpy="0 0 0" />
             <geometry>
@@ -88,5 +86,5 @@
             <inertia ixx="0.001" ixy="0" ixz="0" iyy="0.001" iyz="0" izz="0.001" />
         </inertial>
-        <visual name="Arm_02">
+        <visual>
             <origin xyz="0 0 0" rpy="-1.48894 -1.57209 1.57067" />
             <geometry>
@@ -98,5 +96,5 @@
             </material>
         </visual>
-        <collision name="Arm_02">
+        <collision>
             <origin xyz="-0.00436 0.05688 0.00738" rpy="-1.48879 -1.57209 1.57066" />
             <geometry>
@@ -111,5 +109,5 @@
             <inertia ixx="0.001" ixy="0" ixz="0" iyy="0.001" iyz="0" izz="0.001" />
         </inertial>
-        <visual name="Arm_03">
+        <visual>
             <origin xyz="0 0 0" rpy="1.2416 1.55752 1.5708" />
             <geometry>
@@ -121,5 +119,5 @@
             </material>
         </visual>
-        <collision name="Arm_03.000">
+        <collision>
             <origin xyz="-0.00062 0.00019 0.00049" rpy="1.24161 1.55752 1.5708" />
             <geometry>
@@ -135,5 +133,5 @@
             <inertia ixx="0.001" ixy="0" ixz="0" iyy="0.001" iyz="0" izz="0.001" />
         </inertial>
-        <visual name="Gripper1">
+        <visual>
             <origin xyz="0 -0.01 0.014" rpy="-1.86728 0 0" />
             <geometry>
@@ -145,5 +143,5 @@
             </material>
         </visual>
-        <collision name="Gripper1.000">
+        <collision>
             <origin xyz="0 -0.01 0.014" rpy="-1.86728 0 0" />
             <geometry>
@@ -175,5 +173,5 @@
         </collision>
     </link>
-    <joint name="base_arduino_arm_joint" type="revolute">
+    <joint name="base_waist_joint" type="revolute">
         <origin xyz="-0.00345 -1e-05 0.04449" rpy="0 0 0" />
         <parent link="base_link_arduino_arm" />
@@ -279,15 +277,30 @@
         </actuator>
     </transmission>
-    -->
     <gazebo>
-        <plugin name="gazebo_ros2_control" filename="libgazebo_ros_control.so">
+        <plugin name="gazebo_ros2_control" filename="libgazebo_ros2_control.so">
             <robotNamespace>/</robotNamespace>
         </plugin>
     </gazebo>
+-->
+    <gazebo reference="base_link_arduino_arm">
+        <material>Gazebo/Green</material>
+    </gazebo>
+    <gazebo reference="waist_link">
+        <material>Gazebo/Green</material>
+    </gazebo>
+    <gazebo reference="arm1_link">
+        <material>Gazebo/Green</material>
+    </gazebo>
+    <gazebo reference="arm2_link">
+        <material>Gazebo/Green</material>
+    </gazebo>
+    <gazebo reference="arm3_link">
+        <material>Gazebo/Green</material>
+    </gazebo>
+    <gazebo reference="gripper1_link">
+        <material>Gazebo/Green</material>
+    </gazebo>
     <gazebo reference="gripper2_link">
-    	<material>Gazebo/Green</material>
-	<visual>
-            <transparency>0.25</transparency>
-        </visual>
+        <material>Gazebo/Green</material>
     </gazebo>
 </robot>

Commit message: Use "robot" name, add dummy R/L wheels

File: src/arduino_arm/urdf/arduino_arm.urdf.xacro (robot description, xacro)
@@ -1,8 +1,8 @@
 <?xml version="1.0"?>
-<robot xmlns:xacro="http://www.ros.org/wiki/xacro"  name="arduino_arm">
-<!-- <?xml version="1.0"?> -->
-<!-- created with Phobos 1.0.1 "Capricious Choutengan" -->
-<!-- <robot name="arduino_arm"> -->
-<!-- <link name="base_link"/> -->
+<robot xmlns:xacro="http://www.ros.org/wiki/xacro" name="robot">
+    <!-- <?xml version="1.0"?> -->
+    <!-- created with Phobos 1.0.1 "Capricious Choutengan" -->
+    <!-- <robot name="arduino_arm"> -->
+    <!-- <link name="base_link"/> -->
     <joint name="base_link_arduino_arm_joint" type="fixed">
         <parent link="base_link" />
@@ -160,5 +160,6 @@
             <origin xyz="-0.0015 0.01 -0.0165" rpy="1.25673 0 0" />
             <geometry>
-                <mesh filename="file://$(find arduino_arm)/meshes/gripper2_fix.stl" scale="0.001 0.001 0.001" />
+                <mesh filename="file://$(find arduino_arm)/meshes/gripper2_fix.stl"
+                    scale="0.001 0.001 0.001" />
             </geometry>
             <material name="">
@@ -169,5 +170,5 @@
             <origin xyz="-0.0015 0.01 -0.0165" rpy="1.25673 0 0" />
             <geometry>
-	    	<cylinder length="0.001" radius="0.001"/>
+                <cylinder length="0.001" radius="0.001" />
             </geometry>
         </collision>
@@ -214,5 +215,5 @@
         <axis xyz="0 0 1.0" />
         <limit lower="0" upper="1.047" effort="1000.0" velocity="1.0" />
-	<mimic joint="gripper1_joint" multiplier="1.0" offset="0.0" />
+        <mimic joint="gripper1_joint" multiplier="1.0" offset="0.0" />
     </joint>
     <transmission name="trans_base_joint">

File: src/arduino_arm/urdf/arduino_arm_moveit.urdf.xacro (robot description, xacro)
@@ -1,8 +1,9 @@
 <?xml version="1.0"?>
-<robot xmlns:xacro="http://www.ros.org/wiki/xacro"  name="arduino_arm">
-<!-- <?xml version="1.0"?> -->
-<!-- created with Phobos 1.0.1 "Capricious Choutengan" -->
-<!-- <robot name="arduino_arm"> -->
-    <link name="base_link"/>
+<robot xmlns:xacro="http://www.ros.org/wiki/xacro" name="robot">
+    <xacro:include filename="inertial_macros.xacro" />
+    <!-- <?xml version="1.0"?> -->
+    <!-- created with Phobos 1.0.1 "Capricious Choutengan" -->
+    <!-- <robot name="arduino_arm"> -->
+    <link name="base_link" />
     <joint name="base_link_arduino_arm_joint" type="fixed">
         <parent link="base_link" />
@@ -160,5 +161,6 @@
             <origin xyz="-0.0015 0.01 -0.0165" rpy="1.25673 0 0" />
             <geometry>
-                <mesh filename="file://$(find arduino_arm)/meshes/gripper2_fix.stl" scale="0.001 0.001 0.001" />
+                <mesh filename="file://$(find arduino_arm)/meshes/gripper2_fix.stl"
+                    scale="0.001 0.001 0.001" />
             </geometry>
             <material name="">
@@ -169,5 +171,5 @@
             <origin xyz="-0.0015 0.01 -0.0165" rpy="1.25673 0 0" />
             <geometry>
-	    	<cylinder length="0.001" radius="0.001"/>
+                <cylinder length="0.001" radius="0.001" />
             </geometry>
         </collision>
@@ -214,5 +216,5 @@
         <axis xyz="0 0 1.0" />
         <limit lower="0" upper="1.047" effort="1000.0" velocity="1.0" />
-	<mimic joint="gripper1_joint" multiplier="1.0" offset="0.0" />
+        <mimic joint="gripper1_joint" multiplier="1.0" offset="0.0" />
     </joint>
     <transmission name="trans_base_joint">
@@ -283,4 +285,61 @@
     </gazebo>
 -->
+    <!-- <xacro:property name="wheel_radius" value="0.0001"/>
+    <xacro:property name="wheel_thickness" value="0.026"/>
+    <xacro:property name="wheel_mass" value="0.05"/>
+    <xacro:property name="wheel_offset_y" value="0.1485"/> -->
+    <material name="blue">
+        <color rgba="0.2 0.2 1 1" />
+    </material>
+    <joint name="left_wheel_joint" type="fixed">
+        <parent link="base_link_arduino_arm" />
+        <child link="left_wheel" />
+        <origin xyz="0 0.004 0" rpy="-${pi/2} 0 0" />
+        <axis xyz="0 0 1" />
+    </joint>
+    <link name="left_wheel">
+        <visual>
+            <geometry>
+                <cylinder radius="0.001" length="0.002" />
+            </geometry>
+            <material name="blue" />
+        </visual>
+        <collision>
+            <geometry>
+                <sphere radius="0.001" />
+            </geometry>
+        </collision>
+        <xacro:inertial_cylinder mass="0.003" length="0.002" radius="0.002">
+            <origin xyz="0 0 0" rpy="0 0 0" />
+        </xacro:inertial_cylinder>
+    </link>
+    <gazebo reference="left_wheel">
+        <material>Gazebo/Blue</material>
+    </gazebo>
+    <joint name="right_wheel_joint" type="fixed">
+        <parent link="base_link_arduino_arm" />
+        <child link="right_wheel" />
+        <origin xyz="0 -0.004 0" rpy="${pi/2} 0 0" />
+        <axis xyz="0 0 -1" />
+    </joint>
+    <link name="right_wheel">
+        <visual>
+            <geometry>
+                <cylinder radius="0.001" length="0.002" />
+            </geometry>
+            <material name="blue" />
+        </visual>
+        <collision>
+            <geometry>
+                <sphere radius="0.002" />
+            </geometry>
+        </collision>
+        <xacro:inertial_cylinder mass="0.003" length="0.002" radius="0.001">
+            <origin xyz="0 0 0" rpy="0 0 0" />
+        </xacro:inertial_cylinder>
+    </link>
+    <gazebo reference="right_wheel">
+        <material>Gazebo/Blue</material>
+    </gazebo>
     <gazebo reference="base_link_arduino_arm">
         <material>Gazebo/Green</material>

File: src/arduino_arm_config/config/robot.ros2_control.xacro (robot description, xacro)
@@ -1,7 +1,6 @@
 <?xml version="1.0"?>
 <robot xmlns:xacro="http://www.ros.org/wiki/xacro">
-    <xacro:macro name="arduino_arm_ros2_control" params="name initial_positions_file">
-        <xacro:property name="initial_positions" value="${xacro.load_yaml(initial_positions_file)['initial_positions']}"/>
-        <!-- <ros2_control name="${name}" type="system"> -->
+    <xacro:macro name="robot_ros2_control" params="name initial_positions_file">
+        <xacro:property name="initial_positions" value="${load_yaml(initial_positions_file)['initial_positions']}"/>
         <ros2_control name="${name}" type="system">
             <hardware>

Commit message: Use joint_trajectory for gripper*

File: src/arduino_arm/urdf/arduino_arm.urdf.xacro (robot description, xacro)
@@ -215,5 +215,5 @@
         <axis xyz="0 0 1.0" />
         <limit lower="0" upper="1.047" effort="1000.0" velocity="1.0" />
-        <mimic joint="gripper1_joint" multiplier="1.0" offset="0.0" />
+	    <!-- <mimic joint="gripper1_joint" multiplier="1.0" offset="0.0" /> -->
     </joint>
     <transmission name="trans_base_joint">

File: src/articubot_one/description/ros2_control.xacro (robot description, xacro)
@@ -56,4 +56,11 @@
             </joint>
             <joint name="gripper1_joint">
+              <command_interface name="position">
+                <param name="min">-1</param>
+                <param name="max">1</param>
+              </command_interface>
+              <state_interface name="position"/>
+            </joint>
+            <joint name="gripper2_joint">
               <command_interface name="position">
                 <param name="min">-1</param>
@@ -120,4 +127,11 @@
                 <state_interface name="velocity"/>
             </joint>
+            <joint name="gripper2_joint">
+                <command_interface name="position"/>
+                <state_interface name="position">
+                  <param name="initial_value">0</param>
+                </state_interface>
+                <state_interface name="velocity"/>
+            </joint>
         </ros2_control>
     </xacro:if>
