Commit message: Added chassis_extension

File: src/arduino_arm/urdf/arduino_arm_diy.urdf.xacro (robot description, xacro)
@@ -6,7 +6,7 @@
     <!-- <link name="base_link"/> -->
     <joint name="base_link_arduino_arm_joint" type="fixed">
-        <parent link="base_link" />
+        <parent link="chassis_extension" />
         <child link="base_link_arduino_arm" />
-        <origin xyz="-0.14 0 0.145" rpy="0 0 1.5708" />
+        <origin xyz="0.075 0 0.025" rpy="0 0 -1.5708" />
     </joint>
     <link name="base_link_arduino_arm">
@@ -182,5 +182,5 @@
     </joint>
     <joint name="shoulder_joint" type="revolute">
-        <origin xyz="0.00396 0.01369 0.03521" rpy="1.5708 -0.53778 1.5708" />
+        <origin xyz="0.00396 0.01369 0.03521" rpy="1.5708 -0.02 1.5708" />
         <parent link="waist_link" />
         <child link="arm1_link" />

File: src/articubot_one/description/camera.xacro (robot description, xacro)
@@ -4,5 +4,5 @@
         <parent link="chassis"/>
         <child link="camera_link"/>
-        <origin xyz="0.32 0 0.181" rpy="0 0.18 0"/>
+        <origin xyz="0.30 0 0.181" rpy="0 0.18 0"/>
     </joint>
     <link name="camera_link">

File: src/articubot_one/description/imu.xacro (robot description, xacro)
@@ -4,10 +4,10 @@
         <parent link="chassis" />
         <child link="imu_link" />
-        <origin xyz="0.26 0 0.14" rpy="0 0 0"/>
+        <origin xyz="0.18 0 0.14" rpy="0 0 0"/>
     </joint>
     <link name="imu_link">
         <visual>
             <geometry>
-                <box size="0.025 0.025 0.015" />
+                <box size="0.04 0.04 0.015" />
             </geometry>
             <material name="red"/>

File: src/articubot_one/description/lidar.xacro (robot description, xacro)
@@ -4,5 +4,5 @@
         <parent link="chassis"/>
         <child link="laser_frame"/>
-        <origin xyz="0.20 0 0.212" rpy="0 0 0"/>
+        <origin xyz="0.10 0 0.212" rpy="0 0 0"/>
     </joint>
     <link name="laser_frame">

File: src/articubot_one/description/robot.urdf.xacro (robot description, xacro)
@@ -14,5 +14,5 @@
     <xacro:include filename="imu.xacro" />
     <!-- <xacro:include filename="depth_camera.xacro" /> -->
-    <xacro:include filename="face.xacro" />
+    <!-- <xacro:include filename="face.xacro" /> -->
     <!-- <xacro:include filename="rrbot.urdf.xacro" /> -->
     <!-- <xacro:include filename="$(find robot_arm)/urdf/robot_arm.urdf" /> -->

File: src/articubot_one/description/robot_core.xacro (robot description, xacro)
@@ -5,4 +5,6 @@
     <xacro:property name="chassis_width" value="0.265"/>
     <xacro:property name="chassis_height" value="0.138"/>
+    <xacro:property name="chassis_extension_length" value="0.15"/>
+    <xacro:property name="chassis_extension_height" value="0.01"/>
     <xacro:property name="chassis_mass" value="1.0"/>
     <xacro:property name="wheel_radius" value="0.033"/>
@@ -12,5 +14,5 @@
     <xacro:property name="wheel_offset_y" value="0.1485"/>
     <xacro:property name="wheel_offset_z" value="0.01"/>
-    <xacro:property name="caster_wheel_radius" value="0.01"/>
+    <xacro:property name="caster_wheel_radius" value="0.015"/>
     <xacro:property name="caster_wheel_mass" value="0.01"/>
     <xacro:property name="caster_wheel_offset_x" value="0.075"/>
@@ -81,4 +83,30 @@
         <material>Gazebo/Orange</material>
     </gazebo>
+    <joint name="chassis_extension_joint" type="fixed">
+        <parent link="chassis"/>
+        <child link="chassis_extension"/>
+        <origin xyz="${chassis_length} 0 ${wheel_radius}"/>
+    </joint>
+    <link name="chassis_extension">
+        <visual>
+            <origin xyz="${chassis_extension_length/2} 0 ${chassis_extension_height/2}"/>
+            <geometry>
+                <box size="${chassis_extension_length} ${chassis_width} ${chassis_extension_height}"/>
+            </geometry>
+            <material name="orange"/>
+        </visual>
+        <collision>
+            <origin xyz="${chassis_extension_length/2} 0 ${chassis_extension_height/2}"/>
+            <geometry>
+                <box size="${chassis_extension_length} ${chassis_width} ${chassis_extension_height}"/>
+            </geometry>
+        </collision>
+        <xacro:inertial_box mass="0.01" x="${chassis_extension_length}" y="${chassis_width}" z="${chassis_extension_height}">
+            <origin xyz="${chassis_extension_length/2} 0 ${chassis_extension_height/2}" rpy="0 0 0"/>
+        </xacro:inertial_box>
+    </link>
+    <gazebo reference="chassis_extension">
+        <material>Gazebo/Orange</material>
+    </gazebo>
     <!-- LEFT WHEEL LINK -->
     <joint name="left_wheel_joint" type="continuous">
@@ -144,5 +172,5 @@
                 <sphere radius="${caster_wheel_radius}"/>
             </geometry>
-            <material name="white"/>
+            <material name="blue"/>
         </visual>
         <collision>
@@ -156,5 +184,5 @@
     </link>
     <gazebo reference="caster_wheel">
-        <material>Gazebo/White</material>
+        <material>Gazebo/Blue</material>
         <mu1 value="0.001"/>
         <mu2 value="0.001"/>

Commit message: Configure arm startup position

File: src/arduino_arm/urdf/arduino_arm_diy.urdf.xacro (robot description, xacro)
@@ -182,5 +182,5 @@
     </joint>
     <joint name="shoulder_joint" type="revolute">
-        <origin xyz="0.00396 0.01369 0.03521" rpy="1.5708 -0.02 1.5708" />
+        <origin xyz="0.00396 0.01369 0.03521" rpy="1.5708 -0.022 1.5708" />
         <parent link="waist_link" />
         <child link="arm1_link" />

Commit message: Try to pick up a simple_box

File: src/arduino_arm/urdf/arduino_arm_diy.urdf.xacro (robot description, xacro)
@@ -170,6 +170,10 @@
             <origin xyz="-0.0015 0.01 -0.0165" rpy="1.25673 0 0" />
             <geometry>
+                <mesh filename="file://$(find arduino_arm)/meshes/gripper2_fix.stl"
+                    scale="0.001 0.001 0.001" />
+            </geometry>
+            <!-- <geometry>
                 <cylinder length="0.001" radius="0.001" />
-            </geometry>
+            </geometry> -->
         </collision>
     </link>

File: src/articubot_one/description/ros2_control.xacro (robot description, xacro)
@@ -123,5 +123,5 @@
                 <command_interface name="position"/>
                 <state_interface name="position">
-                  <param name="initial_value">0</param>
+                  <param name="initial_value">0.6</param>
                 </state_interface>
                 <state_interface name="velocity"/>
@@ -130,5 +130,5 @@
                 <command_interface name="position"/>
                 <state_interface name="position">
-                  <param name="initial_value">0</param>
+                  <param name="initial_value">0.6</param>
                 </state_interface>
                 <state_interface name="velocity"/>

Commit message: Model MY robot

File: src/arduino_arm/urdf/arduino_arm_diy.urdf.xacro (robot description, xacro)
@@ -6,7 +6,7 @@
     <!-- <link name="base_link"/> -->
     <joint name="base_link_arduino_arm_joint" type="fixed">
-        <parent link="chassis_extension" />
+        <parent link="chassis" />
         <child link="base_link_arduino_arm" />
-        <origin xyz="0.075 0 0.025" rpy="0 0 -1.5708" />
+        <origin xyz="0.15 0 0.056" rpy="0 0 -1.5708" />
     </joint>
     <link name="base_link_arduino_arm">

File: src/articubot_one/description/camera.xacro (robot description, xacro)
@@ -4,5 +4,5 @@
         <parent link="chassis"/>
         <child link="camera_link"/>
-        <origin xyz="0.30 0 0.181" rpy="0 0.18 0"/>
+        <origin xyz="0.23 0 0.081" rpy="0 0.18 0"/>
     </joint>
     <link name="camera_link">
@@ -14,7 +14,7 @@
         </visual>
         <visual>
-            <origin xyz="0 0 -0.05"/>
+            <origin xyz="0 0 -0.02"/>
             <geometry>
-                <cylinder radius="0.002" length="0.1"/>
+                <cylinder radius="0.002" length="0.06"/>
             </geometry>
             <material name="black"/>

File: src/articubot_one/description/imu.xacro (robot description, xacro)
@@ -4,10 +4,10 @@
         <parent link="chassis" />
         <child link="imu_link" />
-        <origin xyz="0.18 0 0.14" rpy="0 0 0"/>
+        <origin xyz="0.065 0 0.045" rpy="0 0 0"/>
     </joint>
     <link name="imu_link">
         <visual>
             <geometry>
-                <box size="0.04 0.04 0.015" />
+                <box size="0.03 0.03 0.015" />
             </geometry>
             <material name="red"/>

File: src/articubot_one/description/lidar.xacro (robot description, xacro)
@@ -4,5 +4,5 @@
         <parent link="chassis"/>
         <child link="laser_frame"/>
-        <origin xyz="0.10 0 0.212" rpy="0 0 0"/>
+        <origin xyz="0.025 0 0.10" rpy="0 0 0"/>
     </joint>
     <link name="laser_frame">

File: src/articubot_one/description/robot_core.xacro (robot description, xacro)
@@ -2,19 +2,19 @@
 <robot xmlns:xacro="http://www.ros.org/wiki/xacro" >
     <xacro:include filename="inertial_macros.xacro"/>
-    <xacro:property name="chassis_length" value="0.335"/>
-    <xacro:property name="chassis_width" value="0.265"/>
-    <xacro:property name="chassis_height" value="0.138"/>
-    <xacro:property name="chassis_extension_length" value="0.15"/>
-    <xacro:property name="chassis_extension_height" value="0.01"/>
+    <xacro:property name="chassis_length" value="0.25"/>    <!-- 335"/>     -->
+    <xacro:property name="chassis_width" value="0.125"/>    <!-- 265"/>     -->
+    <xacro:property name="chassis_height" value="0.04"/>   <!-- 138"/>     -->
+    <!-- <xacro:property name="chassis_extension_length" value="0.15"/>
+    <xacro:property name="chassis_extension_height" value="0.01"/> -->
     <xacro:property name="chassis_mass" value="1.0"/>
     <xacro:property name="wheel_radius" value="0.033"/>
     <xacro:property name="wheel_thickness" value="0.026"/>
     <xacro:property name="wheel_mass" value="0.05"/>
-    <xacro:property name="wheel_offset_x" value="0.226"/>
-    <xacro:property name="wheel_offset_y" value="0.1485"/>
+    <xacro:property name="wheel_offset_x" value="0.15"/>    <!-- 226"/>     -->
+    <xacro:property name="wheel_offset_y" value="0.09"/>    <!--1485"/>     -->
     <xacro:property name="wheel_offset_z" value="0.01"/>
     <xacro:property name="caster_wheel_radius" value="0.015"/>
     <xacro:property name="caster_wheel_mass" value="0.01"/>
-    <xacro:property name="caster_wheel_offset_x" value="0.075"/>
+    <xacro:property name="caster_wheel_offset_x" value="0.02"/>     <!-- 75"/>      -->
     <xacro:property name="caster_wheel_offset_z" value="${wheel_offset_z - wheel_radius + caster_wheel_radius}"/>
     <material name="white">
@@ -83,5 +83,5 @@
         <material>Gazebo/Orange</material>
     </gazebo>
-    <joint name="chassis_extension_joint" type="fixed">
+    <!-- <joint name="chassis_extension_joint" type="fixed">
         <parent link="chassis"/>
         <child link="chassis_extension"/>
@@ -108,5 +108,5 @@
     <gazebo reference="chassis_extension">
         <material>Gazebo/Orange</material>
-    </gazebo>
+    </gazebo> -->
     <!-- LEFT WHEEL LINK -->
     <joint name="left_wheel_joint" type="continuous">

Commit message: Trying moveit again

File: src/arduino_arm/urdf/arduino_arm_diy.urdf.xacro (robot description, xacro)
@@ -8,5 +8,5 @@
         <parent link="chassis" />
         <child link="base_link_arduino_arm" />
-        <origin xyz="0.15 0 0.056" rpy="0 0 -1.5708" />
+        <origin xyz="0.15 0 0.056" rpy="0 0 0" />
     </joint>
     <link name="base_link_arduino_arm">
@@ -179,5 +179,5 @@
     </link>
     <joint name="base_waist_joint" type="revolute">
-        <origin xyz="-0.00345 -1e-05 0.04449" rpy="0 0 0" />
+        <origin xyz="-0.00345 -1e-05 0.04449" rpy="0 0 -1.5708" />
         <parent link="base_link_arduino_arm" />
         <child link="waist_link" />

File: src/articubot_one_config/config/robot.ros2_control.xacro (robot description, xacro)
@@ -36,11 +36,4 @@
                 <state_interface name="velocity"/>
             </joint>
-            <joint name="gripper1_joint">
-                <command_interface name="position"/>
-                <state_interface name="position">
-                  <param name="initial_value">${initial_positions['gripper1_joint']}</param>
-                </state_interface>
-                <state_interface name="velocity"/>
-            </joint>
         </ros2_control>
     </xacro:macro>

Commit message: Improve robot looks

File: src/arduino_arm/urdf/arduino_arm_diy.urdf.xacro (robot description, xacro)
@@ -8,5 +8,5 @@
         <parent link="chassis" />
         <child link="base_link_arduino_arm" />
-        <origin xyz="0.15 0 0.056" rpy="0 0 0" />
+        <origin xyz="0.18 0 0.056" rpy="0 0 0" />
     </joint>
     <link name="base_link_arduino_arm">

File: src/articubot_one/description/camera.xacro (robot description, xacro)
@@ -9,5 +9,19 @@
         <visual>
             <geometry>
-                <box size="0.010 0.05 0.025"/>
+                <box size="0.010 0.038 0.024"/>
+            </geometry>
+            <material name="black"/>
+        </visual>
+        <visual>
+            <origin xyz="0 0.016 0" rpy="0 ${pi/2} 0"/>
+            <geometry>
+                <cylinder radius="0.0122" length="0.01"/>
+            </geometry>
+            <material name="black"/>
+        </visual>
+        <visual>
+            <origin xyz="0 -0.016 0" rpy="0 ${pi/2} 0"/>
+            <geometry>
+                <cylinder radius="0.0122" length="0.01"/>
             </geometry>
             <material name="black"/>

File: src/articubot_one/description/imu.xacro (robot description, xacro)
@@ -4,5 +4,5 @@
         <parent link="chassis" />
         <child link="imu_link" />
-        <origin xyz="0.065 0 0.045" rpy="0 0 0"/>
+        <origin xyz="0.08 0 0.045" rpy="0 0 0"/>
     </joint>
     <link name="imu_link">

File: src/articubot_one/description/robot_core.xacro (robot description, xacro)
@@ -11,5 +11,5 @@
     <xacro:property name="wheel_thickness" value="0.026"/>
     <xacro:property name="wheel_mass" value="0.05"/>
-    <xacro:property name="wheel_offset_x" value="0.15"/>    <!-- 226"/>     -->
+    <xacro:property name="wheel_offset_x" value="0.18"/>    <!-- 226"/>     -->
     <xacro:property name="wheel_offset_y" value="0.09"/>    <!--1485"/>     -->
     <xacro:property name="wheel_offset_z" value="0.01"/>
