Commit message: arduino_arm works standalone with moveit

File: src/arduino_arm/urdf/arduino_arm_moveit.urdf.xacro (robot description, xacro)
@@ -1,5 +1,4 @@
 <?xml version="1.0"?>
 <robot xmlns:xacro="http://www.ros.org/wiki/xacro" name="robot">
-    <xacro:include filename="inertial_macros.xacro" />
     <!-- <?xml version="1.0"?> -->
     <!-- created with Phobos 1.0.1 "Capricious Choutengan" -->
@@ -9,5 +8,5 @@
         <parent link="base_link" />
         <child link="base_link_arduino_arm" />
-        <origin xyz="-0.14 0 0.145" rpy="0 0 0" />
+        <origin xyz="0.18 0 0.056" rpy="0 0 0" />
     </joint>
     <link name="base_link_arduino_arm">
@@ -171,10 +170,14 @@
             <origin xyz="-0.0015 0.01 -0.0165" rpy="1.25673 0 0" />
             <geometry>
+                <mesh filename="file://$(find arduino_arm)/meshes/gripper2_fix.stl"
+                    scale="0.001 0.001 0.001" />
+            </geometry>
+            <!-- <geometry>
                 <cylinder length="0.001" radius="0.001" />
-            </geometry>
+            </geometry> -->
         </collision>
     </link>
     <joint name="base_waist_joint" type="revolute">
-        <origin xyz="-0.00345 -1e-05 0.04449" rpy="0 0 0" />
+        <origin xyz="-0.00345 -1e-05 0.04449" rpy="0 0 -1.5708" />
         <parent link="base_link_arduino_arm" />
         <child link="waist_link" />
@@ -183,5 +186,5 @@
     </joint>
     <joint name="shoulder_joint" type="revolute">
-        <origin xyz="0.00396 0.01369 0.03521" rpy="1.5708 0.03778 1.5708" />
+        <origin xyz="0.00396 0.01369 0.03521" rpy="1.5708 -0.022 1.5708" />
         <parent link="waist_link" />
         <child link="arm1_link" />
@@ -190,5 +193,5 @@
     </joint>
     <joint name="elbow_joint" type="revolute">
-        <origin xyz="-7e-05 0.11689 -0.00792" rpy="-0.0013 -3.14159 0.03778" />
+        <origin xyz="-7e-05 0.11689 -0.00792" rpy="-0.0013 -3.14159 -1.45" />
         <parent link="arm1_link" />
         <child link="arm2_link" />
@@ -197,5 +200,5 @@
     </joint>
     <joint name="wrist_joint" type="revolute">
-        <origin xyz="-0.0088 0.12752 -0.00487" rpy="-0.01458 3.14159 0" />
+        <origin xyz="-0.0088 0.12752 -0.00487" rpy="-0.01458 3.14159 1.5708" />
         <parent link="arm2_link" />
         <child link="arm3_link" />
@@ -216,5 +219,5 @@
         <axis xyz="0 0 1.0" />
         <limit lower="0" upper="1.047" effort="1000.0" velocity="1.0" />
-        <mimic joint="gripper1_joint" multiplier="1.0" offset="0.0" />
+	    <!-- <mimic joint="gripper1_joint" multiplier="1.0" offset="0.0" /> -->
     </joint>
     <transmission name="trans_base_joint">
@@ -285,63 +288,6 @@
     </gazebo>
 -->
-    <!-- <xacro:property name="wheel_radius" value="0.0001"/>
-    <xacro:property name="wheel_thickness" value="0.026"/>
-    <xacro:property name="wheel_mass" value="0.05"/>
-    <xacro:property name="wheel_offset_y" value="0.1485"/> -->
-    <material name="blue">
-        <color rgba="0.2 0.2 1 1" />
-    </material>
-    <joint name="left_wheel_joint" type="fixed">
-        <parent link="base_link_arduino_arm" />
-        <child link="left_wheel" />
-        <origin xyz="0 0.004 0" rpy="-${pi/2} 0 0" />
-        <axis xyz="0 0 1" />
-    </joint>
-    <link name="left_wheel">
-        <visual>
-            <geometry>
-                <cylinder radius="0.001" length="0.002" />
-            </geometry>
-            <material name="blue" />
-        </visual>
-        <collision>
-            <geometry>
-                <sphere radius="0.001" />
-            </geometry>
-        </collision>
-        <xacro:inertial_cylinder mass="0.003" length="0.002" radius="0.002">
-            <origin xyz="0 0 0" rpy="0 0 0" />
-        </xacro:inertial_cylinder>
-    </link>
-    <gazebo reference="left_wheel">
-        <material>Gazebo/Blue</material>
-    </gazebo>
-    <joint name="right_wheel_joint" type="fixed">
-        <parent link="base_link_arduino_arm" />
-        <child link="right_wheel" />
-        <origin xyz="0 -0.004 0" rpy="${pi/2} 0 0" />
-        <axis xyz="0 0 -1" />
-    </joint>
-    <link name="right_wheel">
-        <visual>
-            <geometry>
-                <cylinder radius="0.001" length="0.002" />
-            </geometry>
-            <material name="blue" />
-        </visual>
-        <collision>
-            <geometry>
-                <sphere radius="0.002" />
-            </geometry>
-        </collision>
-        <xacro:inertial_cylinder mass="0.003" length="0.002" radius="0.001">
-            <origin xyz="0 0 0" rpy="0 0 0" />
-        </xacro:inertial_cylinder>
-    </link>
-    <gazebo reference="right_wheel">
-        <material>Gazebo/Blue</material>
-    </gazebo>
     <gazebo reference="base_link_arduino_arm">
-        <material>Gazebo/Green</material>
+        <material>Gazebo/White</material>
     </gazebo>
     <gazebo reference="waist_link">
@@ -355,11 +301,11 @@
     </gazebo>
     <gazebo reference="arm3_link">
-        <material>Gazebo/Green</material>
+        <material>Gazebo/White</material>
     </gazebo>
     <gazebo reference="gripper1_link">
-        <material>Gazebo/Green</material>
+        <material>Gazebo/White</material>
     </gazebo>
     <gazebo reference="gripper2_link">
-        <material>Gazebo/Green</material>
+        <material>Gazebo/White</material>
     </gazebo>
 </robot>

File: src/arduino_arm_config/config/robot.ros2_control.xacro (robot description, xacro)
@@ -43,4 +43,11 @@
                 <state_interface name="velocity"/>
             </joint>
+            <joint name="gripper2_joint">
+                <command_interface name="position"/>
+                <state_interface name="position">
+                  <param name="initial_value">${initial_positions['gripper2_joint']}</param>
+                </state_interface>
+                <state_interface name="velocity"/>
+            </joint>
         </ros2_control>
     </xacro:macro>

Commit message: Try moveit with planar

File: src/arduino_arm/urdf/arduino_arm_moveit.urdf.xacro (robot description, xacro)
@@ -10,4 +10,20 @@
         <origin xyz="0.18 0 0.056" rpy="0 0 0" />
     </joint>
+    <!--
+    <link name="left_wheel">
+    </link>
+    <joint name="left_wheel_joint" type="fixed">
+        <parent link="base_link" />
+        <child link="left_wheel" />
+        <origin xyz="0 0 0" rpy="0 0 0" />
+    </joint>
+    <link name="right_wheel">
+    </link>
+    <joint name="right_wheel_joint" type="fixed">
+        <parent link="base_link" />
+        <child link="right_wheel" />
+        <origin xyz="0 0 0" rpy="0 0 0" />
+    </joint>
+    -->
     <link name="base_link_arduino_arm">
         <inertial>
