Commit message: Copied arduino_arm_config "stuff" to various files

File: src/arduino_arm_config/config/arduino_arm.ros2_control.xacro (robot description, xacro)
@@ -2,5 +2,6 @@
 <robot xmlns:xacro="http://www.ros.org/wiki/xacro">
     <xacro:macro name="arduino_arm_ros2_control" params="name initial_positions_file">
-        <xacro:property name="initial_positions" value="${load_yaml(initial_positions_file)['initial_positions']}"/>
+        <xacro:property name="initial_positions" value="${xacro.load_yaml(initial_positions_file)['initial_positions']}"/>
+        <!-- <ros2_control name="${name}" type="system"> -->
         <ros2_control name="${name}" type="system">
             <hardware>

File: src/articubot_one/description/robot.urdf.xacro (robot description, xacro)
@@ -19,3 +19,6 @@
     <!-- <xacro:include filename="$(find eezybotarm)/urdf/eezybotarm.urdf.xacro" /> -->
     <xacro:include filename="$(find arduino_arm)/urdf/arduino_arm.urdf.xacro" />
+    <xacro:include filename="$(find arduino_arm_config)/config/arduino_arm.ros2_control.xacro" />
+    <xacro:arg name="initial_positions_file" default="$(find arduino_arm_config)/config/initial_positions.yaml" />
+    <!-- <xacro:arduino_arm_ros2_control name="FakeSystem" initial_positions_file="$(arg initial_positions_file)"/> -->
 </robot>

File: src/articubot_one/description/ros2_control.xacro (robot description, xacro)
@@ -20,7 +20,6 @@
             </joint>
         </ros2_control>
-        <ros2_control name="RealRobotArm" type="system">
+        <!-- <ros2_control name="RealRobotArm" type="system">
             <hardware>
-                <!-- <plugin>gazebo_ros2_control/GazeboSystem</plugin> -->
                 <plugin>ros2_control_demo_example_1/RRBotSystemPositionOnlyHardware</plugin>
                 <param name="example_param_hw_start_duration_sec">0</param>
@@ -28,41 +27,4 @@
                 <param name="example_param_hw_slowdown">100</param>
             </hardware>
-            <!-- <joint name="joint1">
-                <command_interface name="position">
-                    <param name="min">-1</param>
-                    <param name="max">1</param>
-                </command_interface>
-                <state_interface name="position" />
-            </joint>
-            <joint name="joint2">
-                <command_interface name="position">
-                    <param name="min">-1</param>
-                    <param name="max">1</param>
-                </command_interface>
-                <state_interface name="position" />
-            </joint> -->
-        </ros2_control>
-    </xacro:unless>
-    <xacro:if value="$(arg sim_mode)">
-        <ros2_control name="GazeboSystem" type="system">
-            <hardware>
-                <plugin>gazebo_ros2_control/GazeboSystem</plugin>
-            </hardware>
-            <joint name="left_wheel_joint">
-                <command_interface name="velocity">
-                    <param name="min">-10</param>
-                    <param name="max">10</param>
-                </command_interface>
-                <state_interface name="velocity" />
-                <state_interface name="position" />
-            </joint>
-            <joint name="right_wheel_joint">
-                <command_interface name="velocity">
-                    <param name="min">-10</param>
-                    <param name="max">10</param>
-                </command_interface>
-                <state_interface name="velocity" />
-                <state_interface name="position" />
-            </joint>
             <joint name="base_arduino_arm_joint">
                 <command_interface name="position">
@@ -107,4 +69,69 @@
                 <state_interface name="position" />
             </joint>
+        </ros2_control> -->
+    </xacro:unless>
+    <xacro:if value="$(arg sim_mode)">
+        <ros2_control name="GazeboSystem" type="system">
+            <hardware>
+                <plugin>gazebo_ros2_control/GazeboSystem</plugin>
+            </hardware>
+            <joint name="left_wheel_joint">
+                <command_interface name="velocity">
+                    <param name="min">-10</param>
+                    <param name="max">10</param>
+                </command_interface>
+                <state_interface name="velocity" />
+                <state_interface name="position" />
+            </joint>
+            <joint name="right_wheel_joint">
+                <command_interface name="velocity">
+                    <param name="min">-10</param>
+                    <param name="max">10</param>
+                </command_interface>
+                <state_interface name="velocity" />
+                <state_interface name="position" />
+            </joint>
+            <!-- <joint name="base_arduino_arm_joint">
+                <command_interface name="position">
+                    <param name="min">-1</param>
+                    <param name="max">1</param>
+                </command_interface>
+                <state_interface name="position" />
+            </joint>
+            <joint name="shoulder_joint">
+                <command_interface name="position">
+                    <param name="min">-1</param>
+                    <param name="max">1</param>
+                </command_interface>
+                <state_interface name="position" />
+            </joint>
+            <joint name="elbow_joint">
+                <command_interface name="position">
+                    <param name="min">-1</param>
+                    <param name="max">1</param>
+                </command_interface>
+                <state_interface name="position" />
+            </joint>
+            <joint name="wrist_joint">
+                <command_interface name="position">
+                    <param name="min">-1</param>
+                    <param name="max">1</param>
+                </command_interface>
+                <state_interface name="position" />
+            </joint>
+            <joint name="gripper1_joint">
+                <command_interface name="position">
+                    <param name="min">-1</param>
+                    <param name="max">1</param>
+                </command_interface>
+                <state_interface name="position" />
+            </joint>
+            <joint name="gripper2_joint">
+                <command_interface name="position">
+                    <param name="min">-1</param>
+                    <param name="max">1</param>
+                </command_interface>
+                <state_interface name="position" />
+            </joint> -->
         </ros2_control>
     </xacro:if>
@@ -113,5 +140,6 @@
             <parameters>$(find articubot_one)/config/my_controllers.yaml</parameters>
             <parameters>$(find articubot_one)/config/gaz_ros2_ctl_use_sim.yaml</parameters>
-            <parameters>$(find articubot_one)/config/forward_position_publisher.yaml</parameters>
+            <!-- <parameters>$(find arduino_arm_config)/config/ros2_controllers.yaml</parameters> -->
+            <!-- <parameters>$(find articubot_one)/config/forward_position_publisher.yaml</parameters> -->
         </plugin>
     </gazebo>
